File: hardware/Payload_Computer/ICSP.sch (KiCad schematic (older format))
At the start: 1 part

Commit message: Finished ICSP. Added a few leds and filtering caps
Parts:
- added D?: LED, symbol Device:LED
- added R?: 1K, symbol Device:R_US
Connections:
- net labels added: SCK
- wire segments 6 -> 9
Other:
- note added: "THIS LED IS USED TO HELP WITH BOOTLOADER FLASHING AND INITIAL TESTING\n"
Changed lines of the file:
@@
 $Descr A4 11693 8268
 encoding utf-8
-Sheet 10 11
+Sheet 10 13
 Title ""
 Date ""
@@
 $EndComp
 $Comp
-L power:+5V #PWR?
+L power:+5V #PWR0129
 U 1 1 5F8F1BA6
 P 6600 3850
-F 0 "#PWR?" H 6600 3700 50  0001 C CNN
+F 0 "#PWR0129" H 6600 3700 50  0001 C CNN
 F 1 "+5V" V 6615 3978 50  0000 L CNN
 F 2 "" H 6600 3850 50  0001 C CNN
@@
 	6600 3850 6200 3850
 $Comp
-L power:GND #PWR?
+L power:GND #PWR0130
 U 1 1 5F8F270C
 P 6600 4050
-F 0 "#PWR?" H 6600 3800 50  0001 C CNN
+F 0 "#PWR0130" H 6600 3800 50  0001 C CNN
 F 1 "GND" V 6605 3922 50  0000 R CNN
 F 2 "" H 6600 4050 50  0001 C CNN
@@
 Text HLabel 5200 4050 0    50   Input ~ 0
 RESET_1
+$Comp
+L Device:LED D?
+U 1 1 5F985B10
+P 5850 5250
+F 0 "D?" H 5843 5467 50  0000 C CNN
+F 1 "LED" H 5843 5376 50  0000 C CNN
+F 2 "" H 5850 5250 50  0001 C CNN
+F 3 "~" H 5850 5250 50  0001 C CNN
+	1    5850 5250
+	1    0    0    -1
+$EndComp
+$Comp
+L Device:R_US R?
+U 1 1 5F9867EE
+P 6300 5250
+F 0 "R?" V 6095 5250 50  0000 C CNN
+F 1 "1K" V 6186 5250 50  0000 C CNN
+F 2 "" V 6340 5240 50  0001 C CNN
+F 3 "~" H 6300 5250 50  0001 C CNN
+	1    6300 5250
+	0    1    1    0
+$EndComp
+$Comp
+L power:GND #PWR?
+U 1 1 5F986F6F
+P 5200 5250
+F 0 "#PWR?" H 5200 5000 50  0001 C CNN
+F 1 "GND" V 5205 5122 50  0000 R CNN
+F 2 "" H 5200 5250 50  0001 C CNN
+F 3 "" H 5200 5250 50  0001 C CNN
+	1    5200 5250
+	0    1    1    0
+$EndComp
+Wire Wire Line
+	5200 5250 5700 5250
+Wire Wire Line
+	6000 5250 6150 5250
+Wire Wire Line
+	6450 5250 6950 5250
+Text Label 6600 5250 0    50   ~ 0
+SCK
+Text Label 5400 3950 0    50   ~ 0
+SCK
+Text Notes 4650 4850 0    50   ~ 0
+THIS LED IS USED TO HELP WITH BOOTLOADER FLASHING AND INITIAL TESTING\n
 $EndSCHEMATC
