File: hardware/Payload_Computer/ICSP_2.sch (KiCad schematic (older format))
At the start: 1 part

Commit message: Finished ICSP. Added a few leds and filtering caps
Parts:
- added D?: LED, symbol Device:LED
- added R?: 1K, symbol Device:R_US
Connections:
- net labels added: SCK
- wire segments 6 -> 9
Other:
- note added: "THIS LED IS TO HELP WITH BOOTLOADER FLASHING AND INITIAL TESTING\n"
Changed lines of the file:
@@
 $Descr A4 11693 8268
 encoding utf-8
-Sheet 11 11
+Sheet 11 13
 Title ""
 Date ""
@@
 $EndComp
 $Comp
-L power:+5V #PWR?
+L power:+5V #PWR0131
 U 1 1 5F8F455F
 P 6700 3850
-F 0 "#PWR?" H 6700 3700 50  0001 C CNN
+F 0 "#PWR0131" H 6700 3700 50  0001 C CNN
 F 1 "+5V" V 6715 3978 50  0000 L CNN
 F 2 "" H 6700 3850 50  0001 C CNN
@@
 	6700 3850 6300 3850
 $Comp
-L power:GND #PWR?
+L power:GND #PWR0132
 U 1 1 5F8F4566
 P 6700 4050
-F 0 "#PWR?" H 6700 3800 50  0001 C CNN
+F 0 "#PWR0132" H 6700 3800 50  0001 C CNN
 F 1 "GND" V 6705 3922 50  0000 R CNN
 F 2 "" H 6700 4050 50  0001 C CNN
@@
 Text HLabel 5300 4050 0    50   Input ~ 0
 RESET_2
+$Comp
+L Device:LED D?
+U 1 1 5F988B3F
+P 5850 5300
+AR Path="/5F8F06D7/5F988B3F" Ref="D?"  Part="1"
+AR Path="/5F8F071C/5F988B3F" Ref="D?"  Part="1"
+F 0 "D?" H 5843 5517 50  0000 C CNN
+F 1 "LED" H 5843 5426 50  0000 C CNN
+F 2 "" H 5850 5300 50  0001 C CNN
+F 3 "~" H 5850 5300 50  0001 C CNN
+	1    5850 5300
+	1    0    0    -1
+$EndComp
+$Comp
+L Device:R_US R?
+U 1 1 5F988B45
+P 6300 5300
+AR Path="/5F8F06D7/5F988B45" Ref="R?"  Part="1"
+AR Path="/5F8F071C/5F988B45" Ref="R?"  Part="1"
+F 0 "R?" V 6095 5300 50  0000 C CNN
+F 1 "1K" V 6186 5300 50  0000 C CNN
+F 2 "" V 6340 5290 50  0001 C CNN
+F 3 "~" H 6300 5300 50  0001 C CNN
+	1    6300 5300
+	0    1    1    0
+$EndComp
+$Comp
+L power:GND #PWR?
+U 1 1 5F988B4B
+P 5200 5300
+AR Path="/5F8F06D7/5F988B4B" Ref="#PWR?"  Part="1"
+AR Path="/5F8F071C/5F988B4B" Ref="#PWR?"  Part="1"
+F 0 "#PWR?" H 5200 5050 50  0001 C CNN
+F 1 "GND" V 5205 5172 50  0000 R CNN
+F 2 "" H 5200 5300 50  0001 C CNN
+F 3 "" H 5200 5300 50  0001 C CNN
+	1    5200 5300
+	0    1    1    0
+$EndComp
+Wire Wire Line
+	5200 5300 5700 5300
+Wire Wire Line
+	6000 5300 6150 5300
+Wire Wire Line
+	6450 5300 6950 5300
+Text Label 6600 5300 0    50   ~ 0
+SCK
+Text Label 5500 3950 0    50   ~ 0
+SCK
+Text Notes 4650 4900 0    50   ~ 0
+THIS LED IS TO HELP WITH BOOTLOADER FLASHING AND INITIAL TESTING\n
 $EndSCHEMATC
