File: hardware/Payload_Computer/USB_UART2.sch (KiCad schematic (older format))
At the start: 15 parts

Commit message: Finished BNO055
Parts:
- gave numbers to parts that had none: 14
Changed lines of the file:
@@
 $Descr A4 11693 8268
 encoding utf-8
-Sheet 7 17
+Sheet 7 15
 Title ""
 Date ""
@@
 $EndComp
 $Comp
-L Connector:USB_B_Micro J?
+L Connector:USB_B_Micro J2
 U 1 1 5F87457D
 P 3150 3500
-F 0 "J?" H 3207 3967 50  0000 C CNN
+F 0 "J2" H 3207 3967 50  0000 C CNN
 F 1 "USB_B_Micro" H 3207 3876 50  0000 C CNN
 F 2 "" H 3300 3450 50  0001 C CNN
@@
 $EndComp
 $Comp
-L Device:Fuse F?
+L Device:Fuse F2
 U 1 1 5F874583
 P 3850 3300
-F 0 "F?" V 3653 3300 50  0000 C CNN
+F 0 "F2" V 3653 3300 50  0000 C CNN
 F 1 "Fuse" V 3744 3300 50  0000 C CNN
 F 2 "" V 3780 3300 50  0001 C CNN
@@
 	3450 3300 3600 3300
 $Comp
-L Device:CP C?
+L Device:CP C10
 U 1 1 5F87458A
 P 3600 2900
-F 0 "C?" H 3482 2854 50  0000 R CNN
+F 0 "C10" H 3482 2854 50  0000 R CNN
 F 1 "10nF" H 3482 2945 50  0000 R CNN
 F 2 "" H 3638 2750 50  0001 C CNN
@@
 	3600 2750 3600 2550
 $Comp
-L Device:Ferrite_Bead_Small FB?
+L Device:Ferrite_Bead_Small FB2
 U 1 1 5F87459A
 P 4400 3300
-F 0 "FB?" V 4163 3300 50  0000 C CNN
+F 0 "FB2" V 4163 3300 50  0000 C CNN
 F 1 "600 OHM" V 4254 3300 50  0000 C CNN
 F 2 "" V 4330 3300 50  0001 C CNN
@@
 NoConn ~ 8550 3250
 $Comp
-L Device:C C?
+L Device:C C14
 U 1 1 5F8745E7
 P 9550 3450
-F 0 "C?" V 9298 3450 50  0000 C CNN
+F 0 "C14" V 9298 3450 50  0000 C CNN
 F 1 "100nF" V 9389 3450 50  0000 C CNN
 F 2 "" H 9588 3300 50  0001 C CNN
@@
 	10100 3450 9700 3450
 $Comp
-L Device:C C?
+L Device:C C13
 U 1 1 5F8745F0
 P 8900 3000
-F 0 "C?" H 9015 3046 50  0000 L CNN
+F 0 "C13" H 9015 3046 50  0000 L CNN
 F 1 "100nF" H 9015 2955 50  0000 L CNN
 F 2 "" H 8938 2850 50  0001 C CNN
@@
 	8900 2850 8900 2650
 $Comp
-L Device:LED D?
+L Device:LED D4
 U 1 1 5F874606
 P 6850 4950
-F 0 "D?" H 6843 4695 50  0000 C CNN
+F 0 "D4" H 6843 4695 50  0000 C CNN
 F 1 "LED" H 6843 4786 50  0000 C CNN
 F 2 "" H 6850 4950 50  0001 C CNN
@@
 $EndComp
 $Comp
-L Device:LED D?
+L Device:LED D3
 U 1 1 5F87460C
 P 6850 4550
-F 0 "D?" H 6843 4295 50  0000 C CNN
+F 0 "D3" H 6843 4295 50  0000 C CNN
 F 1 "LED" H 6843 4386 50  0000 C CNN
 F 2 "" H 6850 4550 50  0001 C CNN
@@
 	7300 4950 7000 4950
 $Comp
-L Device:R_US R?
+L Device:R_US R5
 U 1 1 5F874618
 P 6300 4550
-F 0 "R?" V 6095 4550 50  0000 C CNN
+F 0 "R5" V 6095 4550 50  0000 C CNN
 F 1 "1K" V 6186 4550 50  0000 C CNN
 F 2 "" V 6340 4540 50  0001 C CNN
@@
 $EndComp
 $Comp
-L Device:R_US R?
+L Device:R_US R6
 U 1 1 5F87461E
 P 6300 4950
-F 0 "R?" V 6095 4950 50  0000 C CNN
+F 0 "R6" V 6095 4950 50  0000 C CNN
 F 1 "1K" V 6186 4950 50  0000 C CNN
 F 2 "" V 6340 4940 50  0001 C CNN
@@
 NoConn ~ 7450 4050
 $Comp
-L Device:R_US R?
+L Device:R_US R7
 U 1 1 5F8E6C6D
 P 6750 3350
-F 0 "R?" V 6545 3350 50  0000 C CNN
+F 0 "R7" V 6545 3350 50  0000 C CNN
 F 1 "1K" V 6636 3350 50  0000 C CNN
 F 2 "" V 6790 3340 50  0001 C CNN
@@
 	8550 3350 9400 3350
 $Comp
-L Device:R_US R?
+L Device:R_US R8
 U 1 1 5F8E8DCF
 P 9800 3050
-F 0 "R?" V 9595 3050 50  0000 C CNN
+F 0 "R8" V 9595 3050 50  0000 C CNN
 F 1 "1K" V 9686 3050 50  0000 C CNN
 F 2 "" V 9840 3040 50  0001 C CNN
@@
 	9950 3050 10200 3050
 $Comp
-L Device:C C?
+L Device:C C12
 U 1 1 5F98A895
 P 4300 5750
-F 0 "C?" H 4415 5796 50  0000 L CNN
+F 0 "C12" H 4415 5796 50  0000 L CNN
 F 1 "100 nF" H 4415 5705 50  0000 L CNN
 F 2 "" H 4338 5600 50  0001 C CNN
@@
 $EndComp
 $Comp
-L Device:CP C?
+L Device:CP C11
 U 1 1 5F98AD93
 P 3850 5750
-F 0 "C?" H 3968 5796 50  0000 L CNN
+F 0 "C11" H 3968 5796 50  0000 L CNN
 F 1 "4.7 uF" H 3968 5705 50  0000 L CNN
 F 2 "" H 3888 5600 50  0001 C CNN
@@
 $EndComp
 $Comp
-L power:+5V #PWR?
+L power:+5V #PWR0135
 U 1 1 5F98B9B9
 P 4050 5200
-F 0 "#PWR?" H 4050 5050 50  0001 C CNN
+F 0 "#PWR0135" H 4050 5050 50  0001 C CNN
 F 1 "+5V" H 4065 5373 50  0000 C CNN
 F 2 "" H 4050 5200 50  0001 C CNN
@@
 Connection ~ 4050 5200
 $Comp
-L power:GND #PWR?
+L power:GND #PWR0136
 U 1 1 5F98E99D
 P 4050 6100
-F 0 "#PWR?" H 4050 5850 50  0001 C CNN
+F 0 "#PWR0136" H 4050 5850 50  0001 C CNN
 F 1 "GND" H 4055 5927 50  0000 C CNN
 F 2 "" H 4050 6100 50  0001 C CNN
