File: hardware/Payload_Computer/Processor 1.sch (KiCad schematic (older format))
At the start: 1 part

Commit message: Added a new processor. Fixed up some libraries. Did some schematic work.
Parts:
- U?: symbol dk_Embedded-Microcontrollers:ATMEGA328P-AU -> Symbols:ATMEGA328P-AU
Changed lines of the file:
@@
 $Descr A4 11693 8268
 encoding utf-8
-Sheet 2 15
+Sheet 2 14
 Title ""
 Date ""
@@
 $EndDescr
 $Comp
-L dk_Embedded-Microcontrollers:ATMEGA328P-AU U?
+L Symbols:ATMEGA328P-AU U?
 U 1 1 5F845D97
 P 6550 3400

Commit message: Minor Changes
Parts:
- U?: symbol Symbols:ATMEGA328P-AU -> Payload_Computer-rescue:ATMEGA328P-AU-Symbols
Changed lines of the file:
@@
 $Descr A4 11693 8268
 encoding utf-8
-Sheet 2 14
+Sheet 2 13
 Title ""
 Date ""
@@
 $EndDescr
 $Comp
-L Symbols:ATMEGA328P-AU U?
+L Payload_Computer-rescue:ATMEGA328P-AU-Symbols U?
 U 1 1 5F845D97
 P 6550 3400
