File: hardware/Payload_Computer/Processor 2.sch (KiCad schematic (older format))
At the start: 1 part

Commit message: Added a new processor. Fixed up some libraries. Did some schematic work.
Parts:
- removed U?: ATMEGA328P-AU, digikey-footprints:TQFP-32_7x7mm, symbol dk_Embedded-Microcontrollers:ATMEGA328P-AU
- added C? (x2): 0.1 uF, symbol Device:C
- added C?: C, symbol Device:C
- added FB? (x2): Ferrite_Bead_Small, symbol Device:Ferrite_Bead_Small
- added R?: 470 OHM, symbol Device:R_US
- added U?: MK20DX256VLH7, QFP50P1200X1200X160-64N, symbol Symbols:MK20DX256VLH7
Connections:
- net labels added: +3.3V, D+, D-, PTA0, PTA1, PTA2, PTA3
- net labels removed: +5V, RXD, TXD
- wire segments 20 -> 39
- no-connect marks 0 -> 3

Commit message: Minor Changes
Parts:
- U?: symbol Symbols:MK20DX256VLH7 -> Payload_Computer-rescue:MK20DX256VLH7-Symbols
Connections:
- net labels added: SCL, SDA
- wire segments 39 -> 41
Changed lines of the file:
@@
 $Descr A4 11693 8268
 encoding utf-8
-Sheet 14 14
+Sheet 14 13
 Title ""
 Date ""
@@
 	2150 3150 2450 3150
 $Comp
-L Symbols:MK20DX256VLH7 U?
+L Payload_Computer-rescue:MK20DX256VLH7-Symbols U?
 U 1 1 5FAEECCE
 P 3550 3850
@@
 Wire Wire Line
 	6850 2000 6850 1800
+Text HLabel 2150 4750 0    50   Input ~ 0
+SCL
+Text HLabel 2150 4850 0    50   Input ~ 0
+SDA
+Wire Wire Line
+	2150 4750 2450 4750
+Wire Wire Line
+	2450 4850 2150 4850
 $EndSCHEMATC
