File: hardware/Payload_Computer/RESET.sch (KiCad schematic (older format))
At the start: 2 parts

Commit message: Added a new processor. Fixed up some libraries. Did some schematic work.
Parts:
- S?: symbol dk_Pushbutton-Switches:GPTS203211B -> Symbols:GPTS203211B
- renumbered R9 to R?
Changed lines of the file:
@@
 $Descr A4 11693 8268
 encoding utf-8
-Sheet 8 15
+Sheet 6 14
 Title ""
 Date ""
@@
 $EndDescr
 $Comp
-L dk_Pushbutton-Switches:GPTS203211B S?
+L Symbols:GPTS203211B S?
 U 1 1 5F8EA95B
 P 5350 3650
@@
 $EndComp
 $Comp
-L power:GND #PWR0125
+L power:GND #PWR?
 U 1 1 5F8EBFC9
 P 4750 3850
-F 0 "#PWR0125" H 4750 3600 50  0001 C CNN
+F 0 "#PWR?" H 4750 3600 50  0001 C CNN
 F 1 "GND" H 4755 3677 50  0000 C CNN
 F 2 "" H 4750 3850 50  0001 C CNN
@@
 $EndComp
 $Comp
-L Device:R_US R9
+L Device:R_US R?
 U 1 1 5F8EC38D
 P 5900 3350
-F 0 "R9" H 5968 3396 50  0000 L CNN
+F 0 "R?" H 5968 3396 50  0000 L CNN
 F 1 "1K" H 5968 3305 50  0000 L CNN
 F 2 "" V 5940 3340 50  0001 C CNN
@@
 $EndComp
 $Comp
-L power:+5V #PWR0126
+L power:+5V #PWR?
 U 1 1 5F8ECA21
 P 5900 3000
-F 0 "#PWR0126" H 5900 2850 50  0001 C CNN
+F 0 "#PWR?" H 5900 2850 50  0001 C CNN
 F 1 "+5V" H 5915 3173 50  0000 C CNN
 F 2 "" H 5900 3000 50  0001 C CNN

Commit message: Minor Changes
Parts:
- S?: symbol Symbols:GPTS203211B -> Payload_Computer-rescue:GPTS203211B-Symbols
Changed lines of the file:
@@
 $Descr A4 11693 8268
 encoding utf-8
-Sheet 6 14
+Sheet 6 13
 Title ""
 Date ""
@@
 $EndDescr
 $Comp
-L Symbols:GPTS203211B S?
+L Payload_Computer-rescue:GPTS203211B-Symbols S?
 U 1 1 5F8EA95B
 P 5350 3650
