File: hardware/Payload_Computer/USB_UART.sch (KiCad schematic (older format))
At the start: 15 parts

Commit message: Finished BNO055
Parts:
- gave numbers to parts that had none: 14
Changed lines of the file:
@@
 $Descr A4 11693 8268
 encoding utf-8
-Sheet 6 17
+Sheet 6 15
 Title ""
 Date ""
@@
 $EndComp
 $Comp
-L Connector:USB_B_Micro J?
+L Connector:USB_B_Micro J1
 U 1 1 5F855AAE
 P 2050 3250
-F 0 "J?" H 2107 3717 50  0000 C CNN
+F 0 "J1" H 2107 3717 50  0000 C CNN
 F 1 "USB_B_Micro" H 2107 3626 50  0000 C CNN
 F 2 "" H 2200 3200 50  0001 C CNN
@@
 $EndComp
 $Comp
-L Device:Fuse F?
+L Device:Fuse F1
 U 1 1 5F856DD3
 P 2750 3050
-F 0 "F?" V 2553 3050 50  0000 C CNN
+F 0 "F1" V 2553 3050 50  0000 C CNN
 F 1 "Fuse" V 2644 3050 50  0000 C CNN
 F 2 "" V 2680 3050 50  0001 C CNN
@@
 	2350 3050 2500 3050
 $Comp
-L Device:CP C?
+L Device:CP C5
 U 1 1 5F857CF6
 P 2500 2650
-F 0 "C?" H 2382 2604 50  0000 R CNN
+F 0 "C5" H 2382 2604 50  0000 R CNN
 F 1 "10nF" H 2382 2695 50  0000 R CNN
 F 2 "" H 2538 2500 50  0001 C CNN
@@
 	2500 2500 2500 2300
 $Comp
-L Device:Ferrite_Bead_Small FB?
+L Device:Ferrite_Bead_Small FB1
 U 1 1 5F85974D
 P 3300 3050
-F 0 "FB?" V 3063 3050 50  0000 C CNN
+F 0 "FB1" V 3063 3050 50  0000 C CNN
 F 1 "600 OHM" V 3154 3050 50  0000 C CNN
 F 2 "" V 3230 3050 50  0001 C CNN
@@
 NoConn ~ 7450 3000
 $Comp
-L Device:C C?
+L Device:C C9
 U 1 1 5F860CEB
 P 8450 3200
-F 0 "C?" V 8198 3200 50  0000 C CNN
+F 0 "C9" V 8198 3200 50  0000 C CNN
 F 1 "100nF" V 8289 3200 50  0000 C CNN
 F 2 "" H 8488 3050 50  0001 C CNN
@@
 	9000 3200 8600 3200
 $Comp
-L Device:C C?
+L Device:C C8
 U 1 1 5F86213C
 P 7800 2750
-F 0 "C?" H 7915 2796 50  0000 L CNN
+F 0 "C8" H 7915 2796 50  0000 L CNN
 F 1 "100nF" H 7915 2705 50  0000 L CNN
 F 2 "" H 7838 2600 50  0001 C CNN
@@
 	7800 2600 7800 2400
 $Comp
-L Device:LED D?
+L Device:LED D2
 U 1 1 5F8654B1
 P 5750 4700
-F 0 "D?" H 5743 4445 50  0000 C CNN
+F 0 "D2" H 5743 4445 50  0000 C CNN
 F 1 "LED" H 5743 4536 50  0000 C CNN
 F 2 "" H 5750 4700 50  0001 C CNN
@@
 $EndComp
 $Comp
-L Device:LED D?
+L Device:LED D1
 U 1 1 5F866842
 P 5750 4300
-F 0 "D?" H 5743 4045 50  0000 C CNN
+F 0 "D1" H 5743 4045 50  0000 C CNN
 F 1 "LED" H 5743 4136 50  0000 C CNN
 F 2 "" H 5750 4300 50  0001 C CNN
@@
 	6200 4700 5900 4700
 $Comp
-L Device:R_US R?
+L Device:R_US R1
 U 1 1 5F868050
 P 5200 4300
-F 0 "R?" V 4995 4300 50  0000 C CNN
+F 0 "R1" V 4995 4300 50  0000 C CNN
 F 1 "1K" V 5086 4300 50  0000 C CNN
 F 2 "" V 5240 4290 50  0001 C CNN
@@
 $EndComp
 $Comp
-L Device:R_US R?
+L Device:R_US R2
 U 1 1 5F868623
 P 5200 4700
-F 0 "R?" V 4995 4700 50  0000 C CNN
+F 0 "R2" V 4995 4700 50  0000 C CNN
 F 1 "1K" V 5086 4700 50  0000 C CNN
 F 2 "" V 5240 4690 50  0001 C CNN
@@
 NoConn ~ 6350 3800
 $Comp
-L Device:R_US R?
+L Device:R_US R3
 U 1 1 5F8E2EB9
 P 5650 3100
-F 0 "R?" V 5445 3100 50  0000 C CNN
+F 0 "R3" V 5445 3100 50  0000 C CNN
 F 1 "1K" V 5536 3100 50  0000 C CNN
 F 2 "" V 5690 3090 50  0001 C CNN
@@
 	7450 3100 8300 3100
 $Comp
-L Device:R_US R?
+L Device:R_US R4
 U 1 1 5F8E4F1C
 P 8600 2750
-F 0 "R?" V 8395 2750 50  0000 C CNN
+F 0 "R4" V 8395 2750 50  0000 C CNN
 F 1 "1K" V 8486 2750 50  0000 C CNN
 F 2 "" V 8640 2740 50  0001 C CNN
@@
 	8750 2750 9000 2750
 $Comp
-L Device:C C?
+L Device:C C7
 U 1 1 5F992766
 P 3050 5800
-F 0 "C?" H 3165 5846 50  0000 L CNN
+F 0 "C7" H 3165 5846 50  0000 L CNN
 F 1 "100 nF" H 3165 5755 50  0000 L CNN
 F 2 "" H 3088 5650 50  0001 C CNN
@@
 $EndComp
 $Comp
-L Device:CP C?
+L Device:CP C6
 U 1 1 5F99276C
 P 2600 5800
-F 0 "C?" H 2718 5846 50  0000 L CNN
+F 0 "C6" H 2718 5846 50  0000 L CNN
 F 1 "4.7 uF" H 2718 5755 50  0000 L CNN
 F 2 "" H 2638 5650 50  0001 C CNN
@@
 $EndComp
 $Comp
-L power:+5V #PWR?
+L power:+5V #PWR0133
 U 1 1 5F992772
 P 2800 5250
-F 0 "#PWR?" H 2800 5100 50  0001 C CNN
+F 0 "#PWR0133" H 2800 5100 50  0001 C CNN
 F 1 "+5V" H 2815 5423 50  0000 C CNN
 F 2 "" H 2800 5250 50  0001 C CNN
@@
 Connection ~ 2800 5250
 $Comp
-L power:GND #PWR?
+L power:GND #PWR0134
 U 1 1 5F99277D
 P 2800 6150
-F 0 "#PWR?" H 2800 5900 50  0001 C CNN
+F 0 "#PWR0134" H 2800 5900 50  0001 C CNN
 F 1 "GND" H 2805 5977 50  0000 C CNN
 F 2 "" H 2800 6150 50  0001 C CNN

Commit message: Added a new processor. Fixed up some libraries. Did some schematic work.
Parts:
- J?: renamed from J1; symbol Connector:USB_B_Micro -> Symbols:USB_B_Micro
- U?: symbol dk_Interface-Controllers:FT232RL-REEL -> Symbols:FT232RL-REEL
- renumbered C5 to C?, C9 to C?, C8 to C?, C7 to C?, C6 to C?, D2 to D?, D1 to D?, F1 to F?, FB1 to FB?, R1 to R?, R2 to R?, R3 to R?, R4 to R?
Changed lines of the file:
@@
 $Descr A4 11693 8268
 encoding utf-8
-Sheet 6 15
+Sheet 5 14
 Title ""
 Date ""
@@
 $EndDescr
 $Comp
-L dk_Interface-Controllers:FT232RL-REEL U?
+L Symbols:FT232RL-REEL U?
 U 1 1 5F852DA8
 P 7050 3000
@@
 $EndComp
 $Comp
-L Connector:USB_B_Micro J1
+L Symbols:USB_B_Micro J?
 U 1 1 5F855AAE
 P 2050 3250
-F 0 "J1" H 2107 3717 50  0000 C CNN
+F 0 "J?" H 2107 3717 50  0000 C CNN
 F 1 "USB_B_Micro" H 2107 3626 50  0000 C CNN
 F 2 "" H 2200 3200 50  0001 C CNN
@@
 $EndComp
 $Comp
-L Device:Fuse F1
+L Device:Fuse F?
 U 1 1 5F856DD3
 P 2750 3050
-F 0 "F1" V 2553 3050 50  0000 C CNN
+F 0 "F?" V 2553 3050 50  0000 C CNN
 F 1 "Fuse" V 2644 3050 50  0000 C CNN
 F 2 "" V 2680 3050 50  0001 C CNN
@@
 	2350 3050 2500 3050
 $Comp
-L Device:CP C5
+L Device:CP C?
 U 1 1 5F857CF6
 P 2500 2650
-F 0 "C5" H 2382 2604 50  0000 R CNN
+F 0 "C?" H 2382 2604 50  0000 R CNN
 F 1 "10nF" H 2382 2695 50  0000 R CNN
 F 2 "" H 2538 2500 50  0001 C CNN
@@
 	2500 3050 2600 3050
 $Comp
-L power:GND #PWR0109
+L power:GND #PWR?
 U 1 1 5F858C58
 P 2500 2300
-F 0 "#PWR0109" H 2500 2050 50  0001 C CNN
+F 0 "#PWR?" H 2500 2050 50  0001 C CNN
 F 1 "GND" H 2505 2127 50  0000 C CNN
 F 2 "" H 2500 2300 50  0001 C CNN
@@
 	2500 2500 2500 2300
 $Comp
-L Device:Ferrite_Bead_Small FB1
+L Device:Ferrite_Bead_Small FB?
 U 1 1 5F85974D
 P 3300 3050
-F 0 "FB1" V 3063 3050 50  0000 C CNN
+F 0 "FB?" V 3063 3050 50  0000 C CNN
 F 1 "600 OHM" V 3154 3050 50  0000 C CNN
 F 2 "" V 3230 3050 50  0001 C CNN
@@
 	2900 3050 3200 3050
 $Comp
-L power:VBUS #PWR0110
+L power:VBUS #PWR?
 U 1 1 5F859D37
 P 3750 3050
-F 0 "#PWR0110" H 3750 2900 50  0001 C CNN
+F 0 "#PWR?" H 3750 2900 50  0001 C CNN
 F 1 "VBUS" V 3765 3178 50  0000 L CNN
 F 2 "" H 3750 3050 50  0001 C CNN
@@
 	3400 3050 3750 3050
 $Comp
-L power:GND #PWR0111
+L power:GND #PWR?
 U 1 1 5F85A3C3
 P 2050 3900
-F 0 "#PWR0111" H 2050 3650 50  0001 C CNN
+F 0 "#PWR?" H 2050 3650 50  0001 C CNN
 F 1 "GND" H 2055 3727 50  0000 C CNN
 F 2 "" H 2050 3900 50  0001 C CNN
@@
 NoConn ~ 2350 3450
 $Comp
-L power:+5V #PWR0112
+L power:+5V #PWR?
 U 1 1 5F85B744
 P 6850 2200
-F 0 "#PWR0112" H 6850 2050 50  0001 C CNN
+F 0 "#PWR?" H 6850 2050 50  0001 C CNN
 F 1 "+5V" H 6865 2373 50  0000 C CNN
 F 2 "" H 6850 2200 50  0001 C CNN
@@
 	6850 2350 6850 2200
 $Comp
-L power:GND #PWR0113
+L power:GND #PWR?
 U 1 1 5F85C222
 P 6850 4500
-F 0 "#PWR0113" H 6850 4250 50  0001 C CNN
+F 0 "#PWR?" H 6850 4250 50  0001 C CNN
 F 1 "GND" H 6855 4327 50  0000 C CNN
 F 2 "" H 6850 4500 50  0001 C CNN
@@
 NoConn ~ 7450 3000
 $Comp
-L Device:C C9
+L Device:C C?
 U 1 1 5F860CEB
 P 8450 3200
-F 0 "C9" V 8198 3200 50  0000 C CNN
+F 0 "C?" V 8198 3200 50  0000 C CNN
 F 1 "100nF" V 8289 3200 50  0000 C CNN
 F 2 "" H 8488 3050 50  0001 C CNN
@@
 	9000 3200 8600 3200
 $Comp
-L Device:C C8
+L Device:C C?
 U 1 1 5F86213C
 P 7800 2750
-F 0 "C8" H 7915 2796 50  0000 L CNN
+F 0 "C?" H 7915 2796 50  0000 L CNN
 F 1 "100nF" H 7915 2705 50  0000 L CNN
 F 2 "" H 7838 2600 50  0001 C CNN
@@
 	7450 2900 7800 2900
 $Comp
-L power:+3.3V #PWR0114
+L power:+3.3V #PWR?
 U 1 1 5F863614
 P 7900 2900
-F 0 "#PWR0114" H 7900 2750 50  0001 C CNN
+F 0 "#PWR?" H 7900 2750 50  0001 C CNN
 F 1 "+3.3V" V 7915 3028 50  0000 L CNN
 F 2 "" H 7900 2900 50  0001 C CNN
@@
 Connection ~ 7800 2900
 $Comp
-L power:GND #PWR0115
+L power:GND #PWR?
 U 1 1 5F8647C2
 P 7800 2400
-F 0 "#PWR0115" H 7800 2150 50  0001 C CNN
+F 0 "#PWR?" H 7800 2150 50  0001 C CNN
 F 1 "GND" H 7805 2227 50  0000 C CNN
 F 2 "" H 7800 2400 50  0001 C CNN
@@
 	7800 2600 7800 2400
 $Comp
-L Device:LED D2
+L Device:LED D?
 U 1 1 5F8654B1
 P 5750 4700
-F 0 "D2" H 5743 4445 50  0000 C CNN
+F 0 "D?" H 5743 4445 50  0000 C CNN
 F 1 "LED" H 5743 4536 50  0000 C CNN
 F 2 "" H 5750 4700 50  0001 C CNN
@@
 $EndComp
 $Comp
-L Device:LED D1
+L Device:LED D?
 U 1 1 5F866842
 P 5750 4300
-F 0 "D1" H 5743 4045 50  0000 C CNN
+F 0 "D?" H 5743 4045 50  0000 C CNN
 F 1 "LED" H 5743 4136 50  0000 C CNN
 F 2 "" H 5750 4300 50  0001 C CNN
@@
 	6200 4700 5900 4700
 $Comp
-L Device:R_US R1
+L Device:R_US R?
 U 1 1 5F868050
 P 5200 4300
-F 0 "R1" V 4995 4300 50  0000 C CNN
+F 0 "R?" V 4995 4300 50  0000 C CNN
 F 1 "1K" V 5086 4300 50  0000 C CNN
 F 2 "" V 5240 4290 50  0001 C CNN
@@
 $EndComp
 $Comp
-L Device:R_US R2
+L Device:R_US R?
 U 1 1 5F868623
 P 5200 4700
-F 0 "R2" V 4995 4700 50  0000 C CNN
+F 0 "R?" V 4995 4700 50  0000 C CNN
 F 1 "1K" V 5086 4700 50  0000 C CNN
 F 2 "" V 5240 4690 50  0001 C CNN
@@
 	5600 4700 5350 4700
 $Comp
-L power:+5V #PWR0116
+L power:+5V #PWR?
 U 1 1 5F869AE2
 P 4600 4500
-F 0 "#PWR0116" H 4600 4350 50  0001 C CNN
+F 0 "#PWR?" H 4600 4350 50  0001 C CNN
 F 1 "+5V" V 4615 4628 50  0000 L CNN
 F 2 "" H 4600 4500 50  0001 C CNN
@@
 NoConn ~ 6350 3800
 $Comp
-L Device:R_US R3
+L Device:R_US R?
 U 1 1 5F8E2EB9
 P 5650 3100
-F 0 "R3" V 5445 3100 50  0000 C CNN
+F 0 "R?" V 5445 3100 50  0000 C CNN
 F 1 "1K" V 5536 3100 50  0000 C CNN
 F 2 "" V 5690 3090 50  0001 C CNN
@@
 	7450 3100 8300 3100
 $Comp
-L Device:R_US R4
+L Device:R_US R?
 U 1 1 5F8E4F1C
 P 8600 2750
-F 0 "R4" V 8395 2750 50  0000 C CNN
+F 0 "R?" V 8395 2750 50  0000 C CNN
 F 1 "1K" V 8486 2750 50  0000 C CNN
 F 2 "" V 8640 2740 50  0001 C CNN
@@
 	8750 2750 9000 2750
 $Comp
-L Device:C C7
+L Device:C C?
 U 1 1 5F992766
 P 3050 5800
-F 0 "C7" H 3165 5846 50  0000 L CNN
+F 0 "C?" H 3165 5846 50  0000 L CNN
 F 1 "100 nF" H 3165 5755 50  0000 L CNN
 F 2 "" H 3088 5650 50  0001 C CNN
@@
 $EndComp
 $Comp
-L Device:CP C6
+L Device:CP C?
 U 1 1 5F99276C
 P 2600 5800
-F 0 "C6" H 2718 5846 50  0000 L CNN
+F 0 "C?" H 2718 5846 50  0000 L CNN
 F 1 "4.7 uF" H 2718 5755 50  0000 L CNN
 F 2 "" H 2638 5650 50  0001 C CNN
@@
 $EndComp
 $Comp
-L power:+5V #PWR0133
+L power:+5V #PWR?
 U 1 1 5F992772
 P 2800 5250
-F 0 "#PWR0133" H 2800 5100 50  0001 C CNN
+F 0 "#PWR?" H 2800 5100 50  0001 C CNN
 F 1 "+5V" H 2815 5423 50  0000 C CNN
 F 2 "" H 2800 5250 50  0001 C CNN
@@
 Connection ~ 2800 5250
 $Comp
-L power:GND #PWR0134
+L power:GND #PWR?
 U 1 1 5F99277D
 P 2800 6150
-F 0 "#PWR0134" H 2800 5900 50  0001 C CNN
+F 0 "#PWR?" H 2800 5900 50  0001 C CNN
 F 1 "GND" H 2805 5977 50  0000 C CNN
 F 2 "" H 2800 6150 50  0001 C CNN

Commit message: Minor Changes
Parts:
- J?: symbol Symbols:USB_B_Micro -> Payload_Computer-rescue:USB_B_Micro-Symbols
- U?: symbol Symbols:FT232RL-REEL -> Payload_Computer-rescue:FT232RL-REEL-Symbols
Changed lines of the file:
@@
 $Descr A4 11693 8268
 encoding utf-8
-Sheet 5 14
+Sheet 5 13
 Title ""
 Date ""
@@
 $EndDescr
 $Comp
-L Symbols:FT232RL-REEL U?
+L Payload_Computer-rescue:FT232RL-REEL-Symbols U?
 U 1 1 5F852DA8
 P 7050 3000
@@
 $EndComp
 $Comp
-L Symbols:USB_B_Micro J?
+L Payload_Computer-rescue:USB_B_Micro-Symbols J?
 U 1 1 5F855AAE
 P 2050 3250
