File: hardware/Payload_Computer/ARDUINO.sch (KiCad schematic (older format))
At the start: 1 part

Commit message: More Library Updates
Parts:
- U?: symbol Payload_Computer-rescue:ATMEGA328P-AU-Symbols -> Symbols:ATMEGA328P-AU
Changed lines of the file:
@@
 $EndDescr
 $Comp
-L Payload_Computer-rescue:ATMEGA328P-AU-Symbols U?
+L Symbols:ATMEGA328P-AU U?
 U 1 1 5F845D97
 P 6550 3400
