File: hardware/Payload_Computer/SERVOS.sch (KiCad schematic (older format))
At the start: 0 parts

Commit message: Minor Changes
Parts:
- added C1001, C1002, C1003, C1004: 0.47 uF, Capacitor_SMD:C_0603_1608Metric_Pad1.08x0.95mm_HandSolder, symbol Device:C
- added C1005, C1006, C1007, C1008: 22 uF, symbol Device:CP
- added J1001, J1002, J1003, J1004: 505567-0381, 505567-0381:5055670381, symbol 505567-0381:505567-0381
- added VR1001, VR1002, VR1003, VR1004: LM2940IMP-5.0_NOPB, LM2940IMP-5:SOT230P700X180-4N, symbol LM2940IMP-5.0_NOPB:LM2940IMP-5.0_NOPB
Connections:
- net labels added: +BATT, GND, SERVO1, SERVO2, SERVO3, SERVO4, SERVO_5V_1, SERVO_5V_2, SERVO_5V_3, SERVO_5V_4
- wire segments 0 -> 60

Commit message: Added some footprints
Parts:
- C1005, C1006, C1007, C1008: footprint (none) -> Capacitor_SMD:C_0603_1608Metric_Pad1.08x0.95mm_HandSolder; Digikey (none) -> 1276-2868-2-ND
Changed lines of the file:
@@
 	5000 1550 5100 1550
 Connection ~ 5100 1550
-Wire Wire Line
-	5000 1250 5500 1250
 $Comp
 L power:GND #PWR01013
@@
 Wire Wire Line
 	5500 1550 5500 1650
-$Comp
-L Device:CP C1005
-U 1 1 602B5EE8
-P 5500 1400
-F 0 "C1005" H 5618 1446 50  0000 L CNN
-F 1 "22 uF" H 5618 1355 50  0000 L CNN
-F 2 "" H 5538 1250 50  0001 C CNN
-F 3 "~" H 5500 1400 50  0001 C CNN
-	1    5500 1400
-	1    0    0    -1
-$EndComp
-Wire Wire Line
-	5500 1250 5950 1250
-Connection ~ 5500 1250
 $Comp
 L 505567-0381:505567-0381 J1001
@@
 	5000 2750 5100 2750
 Connection ~ 5100 2750
-Wire Wire Line
-	5000 2450 5500 2450
 $Comp
 L power:GND #PWR01014
@@
 Wire Wire Line
 	5500 2750 5500 2850
-$Comp
-L Device:CP C1006
-U 1 1 602D94E6
-P 5500 2600
-F 0 "C1006" H 5618 2646 50  0000 L CNN
-F 1 "22 uF" H 5618 2555 50  0000 L CNN
-F 2 "" H 5538 2450 50  0001 C CNN
-F 3 "~" H 5500 2600 50  0001 C CNN
-	1    5500 2600
-	1    0    0    -1
-$EndComp
-Wire Wire Line
-	5500 2450 5950 2450
-Connection ~ 5500 2450
 $Comp
 L 505567-0381:505567-0381 J1002
@@
 	5000 3750 5100 3750
 Connection ~ 5100 3750
-Wire Wire Line
-	5000 3450 5500 3450
 $Comp
 L power:GND #PWR01015
@@
 Wire Wire Line
 	5500 3750 5500 3850
-$Comp
-L Device:CP C1007
-U 1 1 602DCCD5
-P 5500 3600
-F 0 "C1007" H 5618 3646 50  0000 L CNN
-F 1 "22 uF" H 5618 3555 50  0000 L CNN
-F 2 "" H 5538 3450 50  0001 C CNN
-F 3 "~" H 5500 3600 50  0001 C CNN
-	1    5500 3600
-	1    0    0    -1
-$EndComp
-Wire Wire Line
-	5500 3450 5950 3450
-Connection ~ 5500 3450
 $Comp
 L 505567-0381:505567-0381 J1003
@@
 F 0 "C1008" H 5618 4646 50  0000 L CNN
 F 1 "22 uF" H 5618 4555 50  0000 L CNN
-F 2 "" H 5538 4450 50  0001 C CNN
+F 2 "Capacitor_SMD:C_0603_1608Metric_Pad1.08x0.95mm_HandSolder" H 5538 4450 50  0001 C CNN
 F 3 "~" H 5500 4600 50  0001 C CNN
+F 4 "1276-2868-2-ND" H 5500 4600 50  0001 C CNN "Digikey"
 	1    5500 4600
 	1    0    0    -1
@@
 Wire Wire Line
 	6700 4650 7200 4650
+Wire Wire Line
+	5000 3450 5500 3450
+Wire Wire Line
+	5000 2450 5500 2450
+Wire Wire Line
+	5000 1250 5500 1250
+$Comp
+L Device:CP C1007
+U 1 1 602EAC9D
+P 5500 3600
+F 0 "C1007" H 5618 3646 50  0000 L CNN
+F 1 "22 uF" H 5618 3555 50  0000 L CNN
+F 2 "Capacitor_SMD:C_0603_1608Metric_Pad1.08x0.95mm_HandSolder" H 5538 3450 50  0001 C CNN
+F 3 "~" H 5500 3600 50  0001 C CNN
+F 4 "1276-2868-2-ND" H 5500 3600 50  0001 C CNN "Digikey"
+	1    5500 3600
+	1    0    0    -1
+$EndComp
+Connection ~ 5500 3450
+Wire Wire Line
+	5500 3450 5950 3450
+$Comp
+L Device:CP C1006
+U 1 1 602EB28A
+P 5500 2600
+F 0 "C1006" H 5618 2646 50  0000 L CNN
+F 1 "22 uF" H 5618 2555 50  0000 L CNN
+F 2 "Capacitor_SMD:C_0603_1608Metric_Pad1.08x0.95mm_HandSolder" H 5538 2450 50  0001 C CNN
+F 3 "~" H 5500 2600 50  0001 C CNN
+F 4 "1276-2868-2-ND" H 5500 2600 50  0001 C CNN "Digikey"
+	1    5500 2600
+	1    0    0    -1
+$EndComp
+Connection ~ 5500 2450
+Wire Wire Line
+	5500 2450 5950 2450
+$Comp
+L Device:CP C1005
+U 1 1 602EB679
+P 5500 1400
+F 0 "C1005" H 5618 1446 50  0000 L CNN
+F 1 "22 uF" H 5618 1355 50  0000 L CNN
+F 2 "Capacitor_SMD:C_0603_1608Metric_Pad1.08x0.95mm_HandSolder" H 5538 1250 50  0001 C CNN
+F 3 "~" H 5500 1400 50  0001 C CNN
+F 4 "1276-2868-2-ND" H 5500 1400 50  0001 C CNN "Digikey"
+	1    5500 1400
+	1    0    0    -1
+$EndComp
+Connection ~ 5500 1250
+Wire Wire Line
+	5500 1250 5950 1250
 $EndSCHEMATC
