File: hardware/Payload_Computer/FLASH.sch (KiCad schematic (older format))
At the start: 1 part

Commit message: minor changes
Parts:
- gave numbers to parts that had none: 1
Changed lines of the file:
@@
 $EndDescr
 $Comp
-L W25N01GVZEIG_TR:W25N01GVZEIG_TR U?
+L W25N01GVZEIG_TR:W25N01GVZEIG_TR U2001
 U 1 1 603541AA
 P 5950 3450
-F 0 "U?" H 5950 4120 50  0000 C CNN
+F 0 "U2001" H 5950 4120 50  0000 C CNN
 F 1 "W25N01GVZEIG_TR" H 5950 4029 50  0000 C CNN
 F 2 "W25N01GVZEIG_TR:SON127P800X600X80-9N" H 5950 3450 50  0001 L BNN
@@
 $EndComp
 $Comp
-L power:+3.3V #PWR?
+L power:+3.3V #PWR0104
 U 1 1 60354D35
 P 7000 3050
-F 0 "#PWR?" H 7000 2900 50  0001 C CNN
+F 0 "#PWR0104" H 7000 2900 50  0001 C CNN
 F 1 "+3.3V" V 7015 3178 50  0000 L CNN
 F 2 "" H 7000 3050 50  0001 C CNN
@@
 	6850 3050 7000 3050
 $Comp
-L power:GND #PWR?
+L power:GND #PWR0109
 U 1 1 6035554C
 P 7000 3850
-F 0 "#PWR?" H 7000 3600 50  0001 C CNN
+F 0 "#PWR0109" H 7000 3600 50  0001 C CNN
 F 1 "GND" V 7005 3722 50  0000 R CNN
 F 2 "" H 7000 3850 50  0001 C CNN
@@
 	5050 3650 4650 3650
 $Comp
-L power:GND #PWR?
+L power:GND #PWR0110
 U 1 1 6036D706
 P 7000 3650
-F 0 "#PWR?" H 7000 3400 50  0001 C CNN
+F 0 "#PWR0110" H 7000 3400 50  0001 C CNN
 F 1 "GND" V 7005 3522 50  0000 R CNN
 F 2 "" H 7000 3650 50  0001 C CNN
@@
 $EndComp
 $Comp
-L power:GND #PWR?
+L power:GND #PWR0111
 U 1 1 6036D95E
 P 7000 3550
-F 0 "#PWR?" H 7000 3300 50  0001 C CNN
+F 0 "#PWR0111" H 7000 3300 50  0001 C CNN
 F 1 "GND" V 7005 3422 50  0000 R CNN
 F 2 "" H 7000 3550 50  0001 C CNN

Commit message: Minor Changes
Parts:
- added C?: 100nF, Capacitor_SMD:C_0603_1608Metric_Pad1.08x0.95mm_HandSolder, symbol Device:C
Connections:
- net +3V3: now also C?.2
- net GND: now also C?.1
Changed lines of the file:
@@
 $EndComp
 Wire Wire Line
-	6850 3050 7000 3050
+	6850 3050 6900 3050
 $Comp
 L power:GND #PWR0109
@@
 Wire Wire Line
 	7000 3650 6850 3650
+$Comp
+L Device:C C?
+U 1 1 6035BD0E
+P 6900 2900
+F 0 "C?" H 7015 2946 50  0000 L CNN
+F 1 "100nF" H 7015 2855 50  0000 L CNN
+F 2 "Capacitor_SMD:C_0603_1608Metric_Pad1.08x0.95mm_HandSolder" H 6938 2750 50  0001 C CNN
+F 3 "~" H 6900 2900 50  0001 C CNN
+	1    6900 2900
+	1    0    0    -1
+$EndComp
+Connection ~ 6900 3050
+Wire Wire Line
+	6900 3050 7000 3050
+$Comp
+L power:GND #PWR?
+U 1 1 6035C307
+P 6900 2600
+F 0 "#PWR?" H 6900 2350 50  0001 C CNN
+F 1 "GND" V 6905 2472 50  0000 R CNN
+F 2 "" H 6900 2600 50  0001 C CNN
+F 3 "" H 6900 2600 50  0001 C CNN
+	1    6900 2600
+	-1   0    0    1
+$EndComp
+Wire Wire Line
+	6900 2750 6900 2600
 $EndSCHEMATC

Commit message: Annotated a few things
Parts:
- gave numbers to parts that had none: 1
Changed lines of the file:
@@
 	7000 3650 6850 3650
 $Comp
-L Device:C C?
+L Device:C C2001
 U 1 1 6035BD0E
 P 6900 2900
-F 0 "C?" H 7015 2946 50  0000 L CNN
+F 0 "C2001" H 7015 2946 50  0000 L CNN
 F 1 "100nF" H 7015 2855 50  0000 L CNN
 F 2 "Capacitor_SMD:C_0603_1608Metric_Pad1.08x0.95mm_HandSolder" H 6938 2750 50  0001 C CNN
@@
 	6900 3050 7000 3050
 $Comp
-L power:GND #PWR?
+L power:GND #PWR0118
 U 1 1 6035C307
 P 6900 2600
-F 0 "#PWR?" H 6900 2350 50  0001 C CNN
+F 0 "#PWR0118" H 6900 2350 50  0001 C CNN
 F 1 "GND" V 6905 2472 50  0000 R CNN
 F 2 "" H 6900 2600 50  0001 C CNN
