File: hardware/Payload_Computer/LED.sch (KiCad schematic (older format))
At the start: 4 parts

Commit message: minor changes
Parts:
- R1901, R1902, R1903: renamed from R?; footprint (none) -> Resistor_SMD:R_0603_1608Metric_Pad0.98x0.95mm_HandSolder
- gave numbers to parts that had none: 1
Changed lines of the file:
@@
 $EndDescr
 $Comp
-L Device:LED_ABGR D?
+L Device:LED_ABGR D1901
 U 1 1 60334A67
 P 6100 3650
-F 0 "D?" H 6100 4147 50  0000 C CNN
+F 0 "D1901" H 6100 4147 50  0000 C CNN
 F 1 "LED_ABGR" H 6100 4056 50  0000 C CNN
 F 2 "" H 6100 3600 50  0001 C CNN
@@
 $EndComp
 $Comp
-L Device:R_US R?
+L Device:R_US R1901
 U 1 1 60335AE2
 P 5300 3300
-F 0 "R?" V 5095 3300 50  0000 C CNN
+F 0 "R1901" V 5095 3300 50  0000 C CNN
 F 1 "R_US" V 5186 3300 50  0000 C CNN
-F 2 "" V 5340 3290 50  0001 C CNN
+F 2 "Resistor_SMD:R_0603_1608Metric_Pad0.98x0.95mm_HandSolder" V 5340 3290 50  0001 C CNN
 F 3 "~" H 5300 3300 50  0001 C CNN
 	1    5300 3300
@@
 $EndComp
 $Comp
-L Device:R_US R?
+L Device:R_US R1902
 U 1 1 60336395
 P 5300 3650
-F 0 "R?" V 5095 3650 50  0000 C CNN
+F 0 "R1902" V 5095 3650 50  0000 C CNN
 F 1 "R_US" V 5186 3650 50  0000 C CNN
-F 2 "" V 5340 3640 50  0001 C CNN
+F 2 "Resistor_SMD:R_0603_1608Metric_Pad0.98x0.95mm_HandSolder" V 5340 3640 50  0001 C CNN
 F 3 "~" H 5300 3650 50  0001 C CNN
 	1    5300 3650
@@
 $EndComp
 $Comp
-L Device:R_US R?
+L Device:R_US R1903
 U 1 1 603365E3
 P 5300 4000
-F 0 "R?" V 5095 4000 50  0000 C CNN
+F 0 "R1903" V 5095 4000 50  0000 C CNN
 F 1 "R_US" V 5186 4000 50  0000 C CNN
-F 2 "" V 5340 3990 50  0001 C CNN
+F 2 "Resistor_SMD:R_0603_1608Metric_Pad0.98x0.95mm_HandSolder" V 5340 3990 50  0001 C CNN
 F 3 "~" H 5300 4000 50  0001 C CNN
 	1    5300 4000
@@
 $EndComp
 $Comp
-L power:+3.3V #PWR?
+L power:+3.3V #PWR0103
 U 1 1 60336B18
 P 6600 3650
-F 0 "#PWR?" H 6600 3500 50  0001 C CNN
+F 0 "#PWR0103" H 6600 3500 50  0001 C CNN
 F 1 "+3.3V" V 6615 3778 50  0000 L CNN
 F 2 "" H 6600 3650 50  0001 C CNN

Commit message: Added last footprints and started routing
Parts:
- D1901: footprint (none) -> LED:LED
Changed lines of the file:
@@
 F 0 "D1901" H 6100 4147 50  0000 C CNN
 F 1 "LED_ABGR" H 6100 4056 50  0000 C CNN
-F 2 "" H 6100 3600 50  0001 C CNN
+F 2 "LED:LED" H 6100 3600 50  0001 C CNN
 F 3 "~" H 6100 3600 50  0001 C CNN
 	1    6100 3650
