File: hardware/Payload_Computer/SD.sch (KiCad schematic (older format))
At the start: 1 part

Commit message: minor changes
Parts:
- gave numbers to parts that had none: 1
Changed lines of the file:
@@
 $EndDescr
 $Comp
-L 503398-1892:503398-1892 J?
+L 503398-1892:503398-1892 J2102
 U 1 1 6038A9A2
 P 6250 3400
-F 0 "J?" H 6357 4167 50  0000 C CNN
+F 0 "J2102" H 6357 4167 50  0000 C CNN
 F 1 "503398-1892" H 6357 4076 50  0000 C CNN
 F 2 "503398-1892:MOLEX_503398-1892" H 6250 3400 50  0001 L BNN
@@
 $EndComp
 $Comp
-L power:GND #PWR?
+L power:GND #PWR0112
 U 1 1 6038BE8A
 P 7150 4000
-F 0 "#PWR?" H 7150 3750 50  0001 C CNN
+F 0 "#PWR0112" H 7150 3750 50  0001 C CNN
 F 1 "GND" V 7155 3872 50  0000 R CNN
 F 2 "" H 7150 4000 50  0001 C CNN
@@
 	7050 4000 7150 4000
 $Comp
-L power:+3.3V #PWR?
+L power:+3.3V #PWR0113
 U 1 1 6038C540
 P 7150 2900
-F 0 "#PWR?" H 7150 2750 50  0001 C CNN
+F 0 "#PWR0113" H 7150 2750 50  0001 C CNN
 F 1 "+3.3V" V 7165 3028 50  0000 L CNN
 F 2 "" H 7150 2900 50  0001 C CNN

Commit message: Minor Changes
Parts:
- added C?: 100nF, Capacitor_SMD:C_0603_1608Metric_Pad1.08x0.95mm_HandSolder, symbol Device:C
Connections:
- net +3V3: now also C?.2
- net GND: now also C?.1
Changed lines of the file:
@@
 $EndComp
 Wire Wire Line
-	6950 2900 7150 2900
+	6950 2900 7100 2900
 Text HLabel 7150 3200 2    50   Input ~ 0
 SCLK
@@
 NoConn ~ 6950 3400
 NoConn ~ 6950 3700
+$Comp
+L Device:C C?
+U 1 1 6035A6C2
+P 7100 2750
+F 0 "C?" H 7215 2796 50  0000 L CNN
+F 1 "100nF" H 7215 2705 50  0000 L CNN
+F 2 "Capacitor_SMD:C_0603_1608Metric_Pad1.08x0.95mm_HandSolder" H 7138 2600 50  0001 C CNN
+F 3 "~" H 7100 2750 50  0001 C CNN
+	1    7100 2750
+	1    0    0    -1
+$EndComp
+Connection ~ 7100 2900
+Wire Wire Line
+	7100 2900 7150 2900
+$Comp
+L power:GND #PWR?
+U 1 1 6035AD01
+P 7100 2450
+F 0 "#PWR?" H 7100 2200 50  0001 C CNN
+F 1 "GND" V 7105 2322 50  0000 R CNN
+F 2 "" H 7100 2450 50  0001 C CNN
+F 3 "" H 7100 2450 50  0001 C CNN
+	1    7100 2450
+	-1   0    0    1
+$EndComp
+Wire Wire Line
+	7100 2600 7100 2450
 $EndSCHEMATC

Commit message: Annotated a few things
Parts:
- gave numbers to parts that had none: 1
Changed lines of the file:
@@
 NoConn ~ 6950 3700
 $Comp
-L Device:C C?
+L Device:C C2101
 U 1 1 6035A6C2
 P 7100 2750
-F 0 "C?" H 7215 2796 50  0000 L CNN
+F 0 "C2101" H 7215 2796 50  0000 L CNN
 F 1 "100nF" H 7215 2705 50  0000 L CNN
 F 2 "Capacitor_SMD:C_0603_1608Metric_Pad1.08x0.95mm_HandSolder" H 7138 2600 50  0001 C CNN
@@
 	7100 2900 7150 2900
 $Comp
-L power:GND #PWR?
+L power:GND #PWR0119
 U 1 1 6035AD01
 P 7100 2450
-F 0 "#PWR?" H 7100 2200 50  0001 C CNN
+F 0 "#PWR0119" H 7100 2200 50  0001 C CNN
 F 1 "GND" V 7105 2322 50  0000 R CNN
 F 2 "" H 7100 2450 50  0001 C CNN
