File: hardware/Payload_Computer/FANS.sch (KiCad schematic (older format))
At the start: 7 parts, among them J1601 0532610271, J1602 0532610271, J1603 0532610271, J1604 0532610271, Q1601 FDT439

Commit message: More Routing
Parts:
- added C1101: 0.47 uF, Capacitor_SMD:C_0603_1608Metric_Pad1.08x0.95mm_HandSolder, symbol Device:C
- added C1102: 22uF, Capacitor_SMD:C_0603_1608Metric_Pad1.08x0.95mm_HandSolder, symbol Device:C
- added VR1101: LM2940IMP-5.0_NOPB, SOT230P700X180-4N, symbol LM2940IMP-5.0_NOPB:LM2940IMP-5.0_NOPB
Connections:
- net labels added: +BATT
- wire segments 27 -> 37
Changed lines of the file:
@@
 Text Label 7150 4100 0    50   ~ 0
 FANS
+$Comp
+L LM2940IMP-5.0_NOPB:LM2940IMP-5.0_NOPB VR1101
+U 1 1 60377AFA
+P 4550 4050
+F 0 "VR1101" H 4550 4417 50  0000 C CNN
+F 1 "LM2940IMP-5.0_NOPB" H 4550 4326 50  0000 C CNN
+F 2 "SOT230P700X180-4N" H 4550 4050 50  0001 L BNN
+F 3 "" H 4550 4050 50  0001 L BNN
+F 4 "1.80 mm" H 4550 4050 50  0001 L BNN "MAXIMUM_PACKAGE_HEIGHT"
+F 5 "J" H 4550 4050 50  0001 L BNN "PARTREV"
+F 6 "Texas Instruments" H 4550 4050 50  0001 L BNN "MANUFACTURER"
+F 7 "IPC-7351B" H 4550 4050 50  0001 L BNN "STANDARD"
+	1    4550 4050
+	1    0    0    -1
+$EndComp
+$Comp
+L power:+BATT #PWR01101
+U 1 1 603789BE
+P 3700 3950
+F 0 "#PWR01101" H 3700 3800 50  0001 C CNN
+F 1 "+BATT" V 3715 4077 50  0000 L CNN
+F 2 "" H 3700 3950 50  0001 C CNN
+F 3 "" H 3700 3950 50  0001 C CNN
+	1    3700 3950
+	0    -1   -1   0
+$EndComp
+Wire Wire Line
+	3700 3950 3800 3950
+$Comp
+L power:+5V #PWR01105
+U 1 1 603794D8
+P 6100 3950
+F 0 "#PWR01105" H 6100 3800 50  0001 C CNN
+F 1 "+5V" H 6115 4123 50  0000 C CNN
+F 2 "" H 6100 3950 50  0001 C CNN
+F 3 "" H 6100 3950 50  0001 C CNN
+	1    6100 3950
+	0    1    1    0
+$EndComp
+$Comp
+L power:GND #PWR01103
+U 1 1 6037A9EF
+P 5450 4250
+F 0 "#PWR01103" H 5450 4000 50  0001 C CNN
+F 1 "GND" H 5455 4077 50  0000 C CNN
+F 2 "" H 5450 4250 50  0001 C CNN
+F 3 "" H 5450 4250 50  0001 C CNN
+	1    5450 4250
+	0    -1   -1   0
+$EndComp
+Wire Wire Line
+	5250 4250 5350 4250
+Wire Wire Line
+	5250 4150 5350 4150
+Wire Wire Line
+	5350 4150 5350 4250
+Connection ~ 5350 4250
+Wire Wire Line
+	5350 4250 5450 4250
+$Comp
+L Device:C C1101
+U 1 1 6037D852
+P 3800 4100
+F 0 "C1101" H 3915 4146 50  0000 L CNN
+F 1 "0.47 uF" H 3915 4055 50  0000 L CNN
+F 2 "Capacitor_SMD:C_0603_1608Metric_Pad1.08x0.95mm_HandSolder" H 3838 3950 50  0001 C CNN
+F 3 "~" H 3800 4100 50  0001 C CNN
+	1    3800 4100
+	1    0    0    -1
+$EndComp
+Connection ~ 3800 3950
+Wire Wire Line
+	3800 3950 3850 3950
+$Comp
+L power:GND #PWR01102
+U 1 1 6037DDA4
+P 3800 4400
+F 0 "#PWR01102" H 3800 4150 50  0001 C CNN
+F 1 "GND" H 3805 4227 50  0000 C CNN
+F 2 "" H 3800 4400 50  0001 C CNN
+F 3 "" H 3800 4400 50  0001 C CNN
+	1    3800 4400
+	1    0    0    -1
+$EndComp
+Wire Wire Line
+	3800 4400 3800 4250
+$Comp
+L Device:C C1102
+U 1 1 6037EA08
+P 5850 4100
+F 0 "C1102" H 5965 4146 50  0000 L CNN
+F 1 "22uF" H 5965 4055 50  0000 L CNN
+F 2 "Capacitor_SMD:C_0603_1608Metric_Pad1.08x0.95mm_HandSolder" H 5888 3950 50  0001 C CNN
+F 3 "~" H 5850 4100 50  0001 C CNN
+	1    5850 4100
+	1    0    0    -1
+$EndComp
+Wire Wire Line
+	5250 3950 5850 3950
+Connection ~ 5850 3950
+Wire Wire Line
+	5850 3950 6100 3950
+$Comp
+L power:GND #PWR01104
+U 1 1 6037FC41
+P 5850 4400
+F 0 "#PWR01104" H 5850 4150 50  0001 C CNN
+F 1 "GND" H 5855 4227 50  0000 C CNN
+F 2 "" H 5850 4400 50  0001 C CNN
+F 3 "" H 5850 4400 50  0001 C CNN
+	1    5850 4400
+	1    0    0    -1
+$EndComp
+Wire Wire Line
+	5850 4250 5850 4400
 $EndSCHEMATC
