File: hardware/Payload_Computer/Barometer_2.sch (KiCad schematic (older format))
At the start: 0 parts

Commit message: Minor changes
Parts:
- added J?: Conn_01x06_Male, symbol Connector:Conn_01x06_Male
Connections:
- net labels added: +3.3V, CS, GND, MISO, MOSI, SCK
- wire segments 0 -> 6
Changed lines of the file:
@@
 $Descr A4 11693 8268
 encoding utf-8
-Sheet 1 27
+Sheet 26 27
 Title ""
 Date ""
@@
 Comment4 ""
 $EndDescr
+$Comp
+L Connector:Conn_01x06_Male J?
+U 1 1 5FE33A8B
+P 5650 3500
+F 0 "J?" H 5758 3881 50  0000 C CNN
+F 1 "Conn_01x06_Male" H 5758 3790 50  0000 C CNN
+F 2 "" H 5650 3500 50  0001 C CNN
+F 3 "~" H 5650 3500 50  0001 C CNN
+	1    5650 3500
+	1    0    0    -1
+$EndComp
+$Comp
+L power:GND #PWR?
+U 1 1 5FE33F3B
+P 6150 3300
+F 0 "#PWR?" H 6150 3050 50  0001 C CNN
+F 1 "GND" V 6155 3172 50  0000 R CNN
+F 2 "" H 6150 3300 50  0001 C CNN
+F 3 "" H 6150 3300 50  0001 C CNN
+	1    6150 3300
+	0    -1   -1   0
+$EndComp
+$Comp
+L power:+3.3V #PWR?
+U 1 1 5FE34308
+P 6150 3400
+F 0 "#PWR?" H 6150 3250 50  0001 C CNN
+F 1 "+3.3V" V 6165 3528 50  0000 L CNN
+F 2 "" H 6150 3400 50  0001 C CNN
+F 3 "" H 6150 3400 50  0001 C CNN
+	1    6150 3400
+	0    1    1    0
+$EndComp
+Text HLabel 6150 3500 2    50   Input ~ 0
+MOSI
+Text HLabel 6150 3600 2    50   Input ~ 0
+MISO
+Text HLabel 6150 3700 2    50   Input ~ 0
+SCK
+Text HLabel 6150 3800 2    50   Input ~ 0
+CS
+Wire Wire Line
+	5850 3300 6150 3300
+Wire Wire Line
+	6150 3400 5850 3400
+Wire Wire Line
+	5850 3500 6150 3500
+Wire Wire Line
+	6150 3600 5850 3600
+Wire Wire Line
+	5850 3700 6150 3700
+Wire Wire Line
+	6150 3800 5850 3800
 $EndSCHEMATC

Commit message: Finished Fan Schematic. Working on Servos
Parts:
- removed J?: Conn_01x06_Male, symbol Connector:Conn_01x06_Male
- added J2101: 0532610671, 0532610671:MOLEX_0532610671, symbol 0532610671:0532610671
Connections:
- wire segments 6 -> 7
Changed lines of the file:
@@
 $Descr A4 11693 8268
 encoding utf-8
-Sheet 26 26
+Sheet 21 22
 Title ""
 Date ""
@@
 $EndDescr
 $Comp
-L Connector:Conn_01x06_Male J?
-U 1 1 5FE33A8B
-P 5650 3500
-F 0 "J?" H 5758 3881 50  0000 C CNN
-F 1 "Conn_01x06_Male" H 5758 3790 50  0000 C CNN
-F 2 "" H 5650 3500 50  0001 C CNN
-F 3 "~" H 5650 3500 50  0001 C CNN
-	1    5650 3500
-	1    0    0    -1
-$EndComp
-$Comp
-L power:GND #PWR?
+L power:GND #PWR02101
 U 1 1 5FE33F3B
 P 6150 3300
-F 0 "#PWR?" H 6150 3050 50  0001 C CNN
+F 0 "#PWR02101" H 6150 3050 50  0001 C CNN
 F 1 "GND" V 6155 3172 50  0000 R CNN
 F 2 "" H 6150 3300 50  0001 C CNN
@@
 $EndComp
 $Comp
-L power:+3.3V #PWR?
+L power:+3.3V #PWR02102
 U 1 1 5FE34308
 P 6150 3400
-F 0 "#PWR?" H 6150 3250 50  0001 C CNN
+F 0 "#PWR02102" H 6150 3250 50  0001 C CNN
 F 1 "+3.3V" V 6165 3528 50  0000 L CNN
 F 2 "" H 6150 3400 50  0001 C CNN
@@
 Wire Wire Line
 	6150 3800 5850 3800
+$Comp
+L 0532610671:0532610671 J2101
+U 1 1 60295007
+P 5450 3600
+F 0 "J2101" H 5558 4165 50  0000 C CNN
+F 1 "0532610671" H 5558 4074 50  0000 C CNN
+F 2 "0532610671:MOLEX_0532610671" H 5450 3600 50  0001 L BNN
+F 3 "" H 5450 3600 50  0001 L BNN
+F 4 "Molex,LLC" H 5450 3600 50  0001 L BNN "MANUFACTURER"
+	1    5450 3600
+	1    0    0    -1
+$EndComp
+$Comp
+L power:GND #PWR02103
+U 1 1 60295DEF
+P 6150 4000
+F 0 "#PWR02103" H 6150 3750 50  0001 C CNN
+F 1 "GND" V 6155 3872 50  0000 R CNN
+F 2 "" H 6150 4000 50  0001 C CNN
+F 3 "" H 6150 4000 50  0001 C CNN
+	1    6150 4000
+	0    -1   -1   0
+$EndComp
+Wire Wire Line
+	5850 4000 6150 4000
 $EndSCHEMATC
