File: hardware/Payload_Computer/Payload_Computer.kicad_pcb (KiCad board)
At the start: 2 copper layers, 7.6 x 1.3 mm, 91 parts, among them IC901 ZLDO1117G33TA, J1001 505567-0381, J1002 505567-0381, J1003 505567-0381, J1004 505567-0381, J1201 USB3076-XX-X_REVC, J1601 0532610271, J1602 0532610271, J1603 0532610271, J1604 0532610271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

Commit message: Continued all routing
Parts:
- moved J901 84.0 mm to (72.5, 43.2), turned to 90 degrees
- moved Y1 60.1 mm to (260.6, 61.1)
- moved Y2 48.9 mm to (229.6, 61.1)
- moved U801 37.9 mm to (222.6, 65.3), turned to 180 degrees
- moved Y701 11.6 mm to (125.5, 83.9), turned to 180 degrees
- moved D1901 0.19 mm to (161.7, 85.3)
Routing:
- net /PTA1_2: track 0.00 -> 7.21 mm, vias 0 -> 2
- net /PTA2_2: track 0.00 -> 6.07 mm, vias 0 -> 2
- net /XTAL2_1: track 0.00 -> 6.00 mm
- net /XTAL1_1: track 0.00 -> 5.04 mm
- net /PTA0_2: track 0.00 -> 4.05 mm
- net /PTA3_2: track 0.00 -> 3.72 mm
- net Net-(D1901-Pad3): track 0.00 -> 2.68 mm
- net Net-(D1901-Pad2): track 0.00 -> 2.52 mm
- net Net-(C703-Pad2): track 0.00 -> 2.41 mm
- net Net-(C704-Pad2): track 0.00 -> 2.31 mm
- net Net-(D1901-Pad4): track 0.00 -> 2.12 mm

Commit message: Minor Changes
Parts:
- moved R1802 16.9 mm to (97.7, 94.0), turned to 180 degrees
- moved F1801 16.4 mm to (99.0, 88.3), turned to 270 degrees
- moved J1201 14.8 mm to (90.5, 90.4), turned to 270 degrees
- moved FB1801 10.1 mm to (101.8, 88.3), turned to 90 degrees
- moved R1801 8.27 mm to (97.8, 91.4), turned to 180 degrees
- moved C1801 7.73 mm to (96.2, 88.3), turned to 90 degrees
- moved C2202 5.39 mm to (195.2, 76.1)
- moved C2201 5.16 mm to (195.2, 81.6), turned to 180 degrees
- moved U2201 0.93 mm to (195.2, 78.8)
Routing:
- net GND: track 64.8 -> 100.7 mm
- net /XTAL2_2: track 0.00 -> 6.14 mm
- net Net-(C1801-Pad1): track 0.00 -> 5.79 mm
- net Net-(J1201-Pad3): track 0.00 -> 5.63 mm
- net /XTAL1_2: track 0.00 -> 5.11 mm
- net Net-(J1201-Pad2): track 0.00 -> 4.32 mm
- net +3V3: track 0.00 -> 3.99 mm
- net Net-(F1801-Pad1): track 0.00 -> 2.78 mm
Other:
- board size 7.6 x 1.3 mm -> 1.3 x 7.6 mm

Commit message: Did some routing
Parts:
- added C2001: 100nF, Capacitor_SMD:C_0603_1608Metric_Pad1.08x0.95mm_HandSolder, F.Cu at (150.7, 75.6)
- added C2101: 100nF, Capacitor_SMD:C_0603_1608Metric_Pad1.08x0.95mm_HandSolder, F.Cu at (158.6, 75.6)
- moved U1801 149.1 mm to (261.9, 62.6), turned to 180 degrees
- moved F1801 78.9 mm to (135.5, 18.3)
- moved FB1801 78.9 mm to (138.2, 18.3)
- moved J1201 78.9 mm to (127.0, 20.4)
- moved R1802 78.9 mm to (134.2, 24.1)
- moved C1801 78.9 mm to (132.7, 18.3)
- moved R1801 78.9 mm to (134.3, 21.4)
- moved S401 75.5 mm to (250.3, 66.7)
- moved R802 61.3 mm to (134.4, 36.8), turned to 180 degrees
- moved J801 59.7 mm to (127.1, 33.3), turned to 270 degrees
- moved FB2 58.0 mm to (138.3, 31.1), turned to 90 degrees
- moved F2 56.9 mm to (135.5, 31.1), turned to 270 degrees
- moved R801 53.1 mm to (134.4, 34.0), turned to 180 degrees
- moved C10 51.2 mm to (132.7, 31.1), turned to 90 degrees
- moved C704 14.0 mm to (122.8, 80.7)
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Routing:
- net GND: track 100.7 -> 118.8 mm
- net +3V3: track 3.99 -> 19.4 mm
- net /PTA1_1: track 0.00 -> 9.66 mm, vias 0 -> 2
- net /RESET_TEENSY_1: track 0.00 -> 8.00 mm
- net /RESET_1: track 0.00 -> 6.02 mm
- net +BATT: track 9.05 -> 14.9 mm
- net /PTA0_1: track 0.00 -> 5.74 mm, vias 0 -> 2
- net Net-(C10-Pad1): track 0.00 -> 5.74 mm
- net Net-(J801-Pad3): track 0.00 -> 5.59 mm
- net /PTA3_1: track 0.00 -> 4.94 mm
- net /PTA2_1: track 0.00 -> 4.45 mm
- net Net-(J801-Pad2): track 0.00 -> 4.24 mm
- net Net-(C702-Pad2): track 0.00 -> 3.48 mm
- net Net-(C704-Pad2): track 2.31 -> 5.62 mm
- net Net-(C703-Pad2): track 2.41 -> 5.59 mm
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Other:
- outline, holes or cut-outs redrawn

Commit message: More Routing Work
Parts:
- C1701, C1703, C1902, C1904, C601, C602, C901, C903, FB1701, FB1702, FB901, FB902, R1701, R901: moved to B.Cu
- moved Ce 87.2 mm to (258.0, 46.4), turned to 315 degrees
- moved C1703 86.7 mm to (253.9, 51.3), turned to 180 degrees
- moved FB1702 85.5 mm to (253.9, 59.7), turned to 180 degrees
- moved C1902 84.7 mm to (257.9, 54.1), turned to 180 degrees
- moved D1701 83.2 mm to (249.6, 46.1)
- moved R1701 82.3 mm to (253.8, 54.1), turned to 180 degrees
- moved C1904 81.8 mm to (250.3, 54.1)
- moved FB1701 81.2 mm to (253.9, 56.9), turned to 180 degrees
- moved C1701 80.1 mm to (253.9, 62.5)
- moved R1702 76.8 mm to (249.7, 43.3), turned to 180 degrees
- moved C1901 74.1 mm to (244.9, 58.3), turned to 315 degrees
- moved C1702 71.6 mm to (249.7, 63.0), turned to 135 degrees
- moved FB902 34.4 mm to (222.7, 61.4), turned to 180 degrees
- moved R901 34.1 mm to (222.6, 55.6), turned to 180 degrees
- moved S501 34.0 mm to (219.1, 66.7)
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- renumbered C1903 to Ce
Connections:
- C18 pad 1: +5V -> +3V3
- C1901 pad 1: +5V -> +3V3
- C1902 pad 1: +5V -> +3V3
- C1904 pad 1: +5V -> +3V3
- C20 pad 1: +5V -> +3V3
- C601 pad 1: +5V -> +3V3
- C602 pad 1: +5V -> +3V3
- Ce pad 1: +5V -> +3V3
Routing:
- net +3V3: track 19.4 -> 65.4 mm, vias 0 -> 6
- net Net-(C1701-Pad1): track 0.00 -> 18.7 mm, vias 0 -> 2
- net Net-(C901-Pad1): track 0.00 -> 17.1 mm, vias 0 -> 2
- net /RESET_TEENSY_2: track 0.00 -> 16.6 mm, vias 0 -> 3
- net Net-(C1702-Pad2): track 0.00 -> 13.9 mm, vias 0 -> 1
- net Net-(C902-Pad2): track 0.00 -> 12.3 mm, vias 0 -> 1
- net Net-(C1703-Pad1): track 0.00 -> 10.4 mm, vias 0 -> 1
- net Net-(C903-Pad1): track 0.00 -> 9.91 mm, vias 0 -> 1
- net /RESET_2: track 0.00 -> 6.34 mm
- net Net-(C901-Pad2): track 0.00 -> 4.60 mm, vias 0 -> 1
- net Net-(D901-Pad1): track 0.00 -> 2.90 mm
- net Net-(C1701-Pad2): track 0.00 -> 2.84 mm, vias 0 -> 1
- net /SCK: track 0.00 -> 2.70 mm

Commit message: Updated LED. Need to fix Mosfet footprint
Parts:
- C2101: moved to B.Cu
- moved R1901 86.6 mm to (238.5, 47.2), turned to 180 degrees
- moved D1901 85.0 mm to (239.4, 50.8), turned to 180 degrees
- moved R1902 79.1 mm to (234.2, 47.2), turned to 180 degrees
- moved R1903 73.4 mm to (233.0, 50.8), turned to 180 degrees
- moved C2101 16.3 mm to (143.4, 69.6), turned to 180 degrees
- moved C2001 12.0 mm to (155.3, 86.7), turned to 90 degrees
- renumbered Ce to C1903
Connections:
- net Net-(U1701-Pad35) renamed /TEENSY3.2_1/LED_RED
- net Net-(U1701-Pad36) renamed /TEENSY3.2_1/LED_BLUE
- net Net-(U1701-Pad37) renamed /TEENSY3.2_1/LED_GREEN
- U901 pad 35: Net-(U901-Pad35) -> /LED_BLUE
- U901 pad 36: Net-(U901-Pad36) -> /LED_RED
- U901 pad 37: Net-(U901-Pad37) -> /LED_GREEN
Routing:
- net /LED_RED: track 0.00 -> 11.7 mm, vias 0 -> 2
- net /LED_GREEN: track 0.00 -> 7.37 mm
- net +5V: track 0.00 -> 6.30 mm
- net +3V3: track 65.4 -> 71.6 mm, vias 6 -> 7
- net /LED_BLUE: track 0.00 -> 4.29 mm

Commit message: More Routing
Parts:
- added C1101: 0.47 uF, Capacitor_SMD:C_0603_1608Metric_Pad1.08x0.95mm_HandSolder, F.Cu at (103.0, 55.3)
- added C1102: 22uF, Capacitor_SMD:C_0603_1608Metric_Pad1.08x0.95mm_HandSolder, F.Cu at (103.0, 59.8)
- added VR1101: LM2940IMP-5.0_NOPB, LM2940IMP-5:SOT230P700X180-4N, F.Cu at (108.8, 58.4)
- C10, C1801, F1801, F2, FB1801, FB2, R1702, R902: moved to B.Cu
- moved J1003 177.5 mm to (241.4, 93.3), turned to 270 degrees
- moved C1007 172.1 mm to (235.2, 88.7), turned to 180 degrees
- moved C1004 167.0 mm to (235.1, 97.8), turned to 180 degrees
- moved VR1003 166.5 mm to (232.9, 93.2), turned to 180 degrees
- moved C1005 163.7 mm to (208.4, 97.8), turned to 0 degrees
- moved VR1001 158.9 mm to (210.7, 93.2), turned to 0 degrees
- moved J1001 154.7 mm to (202.2, 93.2), turned to 90 degrees
- moved C1002 151.7 mm to (208.4, 88.6), turned to 0 degrees
- moved J1004 143.3 mm to (241.4, 69.5), turned to 270 degrees
- moved C1008 138.7 mm to (235.2, 65.0), turned to 180 degrees
- moved VR1004 132.7 mm to (233.0, 69.5), turned to 180 degrees
- moved C1001 132.6 mm to (235.2, 74.1), turned to 180 degrees
- moved C1006 128.2 mm to (208.3, 74.1), turned to 0 degrees
- moved VR1002 123.8 mm to (210.6, 69.5), turned to 0 degrees
- moved J1002 118.7 mm to (202.1, 69.5), turned to 90 degrees
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Connections:
- net /D+_1 renamed /D1_+
- net /D+_2 renamed /D2_+
- net /D-_1 renamed /D1_-
- net /D-_2 renamed /D2_-
Routing:
- net /SERVO3: track 0.00 -> 33.4 mm
- net /PTA1_1: track 9.66 -> 37.4 mm, vias 2 -> 5
- net /SERVO1: track 0.00 -> 25.4 mm, vias 0 -> 2
- net /PTA1_2: track 9.34 -> 34.3 mm, vias 2 -> 5
- net /SERVO2: track 0.00 -> 17.5 mm, vias 0 -> 2
- net /SERVO4: track 0.00 -> 15.6 mm
- net /D2_-: track 0.00 -> 15.0 mm, vias 0 -> 2
- net /D2_+: track 0.00 -> 15.0 mm
- net /D1_+: track 0.00 -> 14.3 mm
- net /D1_-: track 0.00 -> 14.3 mm, vias 0 -> 2
- net /RESET_TEENSY_1: track 8.00 -> 17.4 mm, vias 0 -> 3
- net Net-(C1701-Pad1): track 18.7 -> 25.6 mm, vias 2 -> 1
- net GND: track 118.8 -> 125.0 mm
- net /TEENSY3.2_1/SCK: track 0.00 -> 5.38 mm
- net Net-(D1701-Pad1): track 0.00 -> 4.52 mm, vias 0 -> 1
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Other:
- board size 1.3 x 7.6 mm -> 50 x 60 mm

Commit message: Did some more routing. Need to really work on condensing some things
Parts:
- C2101: moved to F.Cu
- J2102: moved to B.Cu
- moved J901 142.4 mm to (213.4, 64.3)
- moved C1008 118.2 mm to (135.6, 128.7)
- moved J1004 118.2 mm to (141.9, 133.3)
- moved VR1004 118.2 mm to (133.4, 133.3)
- moved C1001 118.2 mm to (135.7, 137.9)
- moved C1007 102.8 mm to (135.6, 114.3)
- moved J1003 102.8 mm to (141.8, 118.9)
- moved VR1003 102.8 mm to (133.3, 118.9)
- moved C1004 102.8 mm to (135.6, 123.4)
- moved C1005 92.9 mm to (132.0, 44.9)
- moved VR1001 92.9 mm to (134.2, 40.3)
- moved C1002 92.9 mm to (131.9, 35.8)
- moved J1001 92.9 mm to (125.7, 40.4)
- moved C1003 61.7 mm to (154.2, 35.2)
- moved C1006 61.7 mm to (154.2, 44.4)
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Routing:
- net /SERVO3: track 33.4 -> 0.00 mm
- net /SERVO1: track 25.4 -> 0.00 mm, vias 2 -> 0
- net /SERVO2: track 17.5 -> 0.00 mm, vias 2 -> 0
- net /SERVO4: track 15.6 -> 6.19 mm
- net GND: track 125.0 -> 132.4 mm
- added copper zone on +3.3V, net +3V3
- added copper zone on B.Cu, net GND
- added copper zone on F.Cu, net GND
- added copper zone on GND, net GND
Other:
- copper layers 2 -> 4

Commit message: More Changes
Parts:
- added C1009: 0.47 uF, Capacitor_SMD:C_0603_1608Metric_Pad1.08x0.95mm_HandSolder, F.Cu at (121.6, 38.2)
- added C1010: 0.47 uF, Capacitor_SMD:C_0603_1608Metric_Pad1.08x0.95mm_HandSolder, F.Cu at (121.6, 51.6)
- added C1011: 22 uF, Capacitor_SMD:C_0603_1608Metric_Pad1.08x0.95mm_HandSolder, F.Cu at (121.6, 29.2)
- added C1012: 22 uF, Capacitor_SMD:C_0603_1608Metric_Pad1.08x0.95mm_HandSolder, F.Cu at (121.6, 42.5)
- added J1005: 505567-0381, 505567-0381:5055670381, F.Cu at (127.9, 33.8)
- added J1006: 505567-0381, 505567-0381:5055670381, F.Cu at (127.8, 47.0)
- added VR1005: LM2940IMP-5.0_NOPB, LM2940IMP-5:SOT230P700X180-4N, F.Cu at (119.3, 33.8)
- added VR1006: LM2940IMP-5.0_NOPB, LM2940IMP-5:SOT230P700X180-4N, F.Cu at (119.3, 47.1)
- moved J1001 108.0 mm to (123.7, 148.3)
- moved J1002 108.0 mm to (146.0, 147.7)
- moved VR1001 108.0 mm to (132.2, 148.3)
- moved C1002 108.0 mm to (129.9, 143.7)
- moved C1003 108.0 mm to (152.2, 143.2)
- moved C1005 108.0 mm to (129.9, 152.9)
- moved C1006 108.0 mm to (152.1, 152.3)
- moved VR1002 108.0 mm to (154.4, 147.7)
- moved C1004 100.8 mm to (121.6, 23.6)
- moved J1003 100.8 mm to (127.8, 19.1)
- moved VR1003 100.8 mm to (119.4, 19.1)
- moved C1007 100.8 mm to (121.6, 14.5)
- moved C904 73.3 mm to (233.7, 72.3)
- moved C905 73.3 mm to (233.7, 68.1)
- moved D902 73.3 mm to (231.4, 72.1)
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Connections:
- U901 pad 62: /TEENSY 3.2_2/PWM1 -> /SERVO5
- U901 pad 63: /TEENSY 3.2_2/PWM2 -> /SERVO6
Routing:
- net GND: track 132.4 -> 170.5 mm
- net /SERVOS/SERVO_5V_4: track 6.25 -> 18.9 mm
- net +3V3: track 71.6 -> 65.4 mm, vias 7 -> 6
- net +BATT: track 17.6 -> 22.1 mm
