File: hardware/Payload_Computer/Payload_Computer.kicad_pcb (KiCad board)
At the start: 4 copper layers, 50 x 60 mm, 104 parts, among them IC901 ZLDO1117G33TA, J1001 505567-0381, J1002 505567-0381, J1003 505567-0381, J1004 505567-0381, J1005 505567-0381, J1006 505567-0381, J1201 USB3076-XX-X_REVC, J1601 0532610271, J1602 0532610271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

Commit message: More Routing
Parts:
- added H101: MountingHole, MountingHole:MountingHole_3.2mm_M3, F.Cu at (260.6, 45.4)
- added H102: MountingHole, MountingHole:MountingHole_3.2mm_M3, F.Cu at (260.9, 36.1)
- added H103: MountingHole, MountingHole:MountingHole_3.2mm_M3, F.Cu at (268.9, 36.1)
- added H104: MountingHole, MountingHole:MountingHole_3.2mm_M3, F.Cu at (276.8, 36.1)
- C1009, C1010, C1011, C1012, C1101, C1102, C2001, C2101, C702, C703, C704, D1601, Q1601, R1601, R701, R702, R703, U701, VR1005, VR1006, VR1101, Y701: moved to B.Cu
- moved C1004 144.2 mm to (234.9, 112.8)
- moved J1003 144.2 mm to (241.1, 108.3)
- moved C1007 144.2 mm to (234.9, 103.7)
- moved VR1003 144.2 mm to (232.7, 108.3)
- moved C1009 142.2 mm to (233.7, 125.7), turned to 90 degrees
- moved VR1005 141.9 mm to (229.2, 123.4), turned to 90 degrees
- moved J1005 141.3 mm to (229.2, 132.2), turned to 180 degrees
- moved C1011 141.2 mm to (224.7, 125.7), turned to 90 degrees
- moved J1604 139.2 mm to (239.2, 98.6), turned to 90 degrees
- moved J1602 136.2 mm to (239.2, 89.2), turned to 90 degrees
- moved C1010 123.5 mm to (220.4, 125.7), turned to 90 degrees
- moved VR1006 123.1 mm to (215.9, 123.4), turned to 90 degrees
- moved J1006 122.4 mm to (215.9, 132.2), turned to 180 degrees
- moved C1012 122.3 mm to (211.3, 125.7), turned to 90 degrees
- moved C1101 111.6 mm to (210.7, 84.5)
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Connections:
- net /TEENSY 3.2_2/PWM4 renamed Net-(U901-Pad45)
- net Net-(U1701-Pad38) renamed /TEENSY3.2_1/SD_FLASH
- net Net-(U1701-Pad41) renamed /TEENSY3.2_1/FLASH_CS
- J2101 pad 3: /Barometer/Barometer_2/MOSI -> /MOSI
- J2101 pad 4: /Barometer/Barometer_2/MISO -> /MISO
- J2101 pad 5: /Barometer/Barometer_2/SCK -> /SCK
- J2101 pad 6: /Barometer/Barometer_2/CS -> /CS_BARO2
- U1701 pad 45: /SERVO4 -> Net-(U1701-Pad45)
- U1701 pad 64: Net-(U1701-Pad64) -> /SERVO4
- U901 pad 38: Net-(U901-Pad38) -> /CS_SD
- U901 pad 41: Net-(U901-Pad41) -> /CS_FLASH
- U901 pad 44: /TEENSY 3.2_2/PWM3 -> /CS_BARO
- U901 pad 64: Net-(U901-Pad64) -> /CS_BARO2
Routing:
- net +BATT: track 22.1 -> 311.4 mm, vias 0 -> 8
- net GND: track 170.5 -> 262.7 mm, vias 0 -> 25
- net /SERVO4: track 6.19 -> 65.3 mm, vias 0 -> 2
- net VBUS: track 0.00 -> 57.7 mm, vias 0 -> 3
- net /FANS/FANS: track 0.00 -> 57.2 mm, vias 0 -> 2
- net /SCK: track 6.49 -> 63.6 mm, vias 0 -> 4
- net /FANS: track 0.00 -> 55.3 mm, vias 0 -> 1
- net /MISO: track 2.93 -> 56.5 mm, vias 0 -> 2
- net /MOSI: track 3.33 -> 56.8 mm, vias 0 -> 4
- net /SERVO6: track 0.00 -> 45.7 mm, vias 0 -> 4
- net +3V3: track 65.4 -> 91.7 mm, vias 6 -> 23
- net /SERVO2: track 0.00 -> 25.5 mm, vias 0 -> 2
- net /CS_BARO: track 0.00 -> 21.2 mm
- net /CS_FLASH: track 0.00 -> 17.3 mm, vias 0 -> 2
- net /CS_BARO2: track 0.00 -> 17.3 mm
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Other:
- outline, holes or cut-outs redrawn
