File: hardware/Payload_Computer/Barometer.sch (KiCad schematic (older format))
At the start: 0 parts

Commit message: Minor changes
Connections:
- net labels added: CS_BARO2, MISO, MOSI
- net labels removed: SDI, SDO
- wire segments 4 -> 8
Changed lines of the file:
@@
 F0 "Barometer_2" 50
 F1 "Barometer_2.sch" 50
+F2 "MOSI" I R 9160 3150 50
+F3 "MISO" I R 9160 3300 50
+F4 "SCK" I R 9160 3450 50
+F5 "CS" I R 9160 3600 50
 $EndSheet
 Wire Wire Line
@@
 Wire Wire Line
 	2220 4160 1620 4160
-Text Label 1770 3300 0    50   ~ 0
-SDO
-Text Label 1770 3590 0    50   ~ 0
-SCK
-Text Label 1780 3870 0    50   ~ 0
-SDI
-Text Label 1780 4160 0    50   ~ 0
-CSB
 Text HLabel 1620 3300 0    50   Input ~ 0
-SDO
+MISO
 Text HLabel 1620 3590 0    50   Input ~ 0
 SCK
 Text HLabel 1620 3870 0    50   Input ~ 0
-SDI
+MOSI
 Text HLabel 1620 4160 0    50   Input ~ 0
 CSB
@@
 F0 "Barometer_1" 50
 F1 "Barometer_1.sch" 50
-F2 "SDO" I L 2220 3300 50
-F3 "SCK" I L 2220 3590 50
-F4 "SDI" I L 2220 3870 50
-F5 "CSB" I L 2220 4160 50
+F2 "SCK" I L 2220 3590 50
+F3 "CSB" I L 2220 4160 50
+F4 "MISO" I L 2220 3300 50
+F5 "MOSI" I L 2220 3870 50
 $EndSheet
+Wire Wire Line
+	9150 3150 10050 3150
+Wire Wire Line
+	9150 3300 10050 3300
+Wire Wire Line
+	9150 3450 10050 3450
+Text HLabel 10050 3600 2    50   Input ~ 0
+CS_BARO2
+Wire Wire Line
+	9150 3600 10050 3600
+Text Label 9500 3150 0    50   ~ 0
+MOSI
+Text Label 9500 3300 0    50   ~ 0
+MISO
+Text Label 9500 3450 0    50   ~ 0
+SCK
+Text Label 1850 3870 0    50   ~ 0
+MOSI
+Text Label 1850 3590 0    50   ~ 0
+SCK
+Text Label 1870 3300 0    50   ~ 0
+MISO
 $EndSCHEMATC

Commit message: More Changes
Changed lines of the file:
@@
 Text Label 1870 3300 0    50   ~ 0
 MISO
+Text HLabel 10050 3300 2    50   Input ~ 0
+MISO
+Text HLabel 10050 3150 2    50   Input ~ 0
+MOSI
+Text HLabel 10050 3450 2    50   Input ~ 0
+SCK
 $EndSCHEMATC

Commit message: More Routing
Connections:
- net labels added: MISO_2, MOSI_2, SCK_2
Changed lines of the file:
@@
 F5 "MOSI" I L 2220 3870 50
 $EndSheet
-Wire Wire Line
-	9150 3150 10050 3150
-Wire Wire Line
-	9150 3300 10050 3300
-Wire Wire Line
-	9150 3450 10050 3450
 Text HLabel 10050 3600 2    50   Input ~ 0
 CS_BARO2
-Wire Wire Line
-	9150 3600 10050 3600
-Text Label 9500 3150 0    50   ~ 0
-MOSI
-Text Label 9500 3300 0    50   ~ 0
-MISO
-Text Label 9500 3450 0    50   ~ 0
-SCK
 Text Label 1850 3870 0    50   ~ 0
 MOSI
@@
 Text Label 1870 3300 0    50   ~ 0
 MISO
+Text HLabel 10050 3150 2    50   Input ~ 0
+MOSI_2
+Text HLabel 10050 3450 2    50   Input ~ 0
+SCK_2
 Text HLabel 10050 3300 2    50   Input ~ 0
-MISO
-Text HLabel 10050 3150 2    50   Input ~ 0
-MOSI
-Text HLabel 10050 3450 2    50   Input ~ 0
-SCK
+MISO_2
+Wire Wire Line
+	9160 3300 10050 3300
+Wire Wire Line
+	10050 3150 9160 3150
+Wire Wire Line
+	10050 3450 9160 3450
+Wire Wire Line
+	10050 3600 9160 3600
 $EndSCHEMATC
