File: hardware/Payload_Computer/Payload_Computer.sch (KiCad schematic (older format))
At the start: 0 parts

Commit message: More Routing
Parts:
- added H101, H102, H103, H104: MountingHole, MountingHole:MountingHole_3.2mm_M3, symbol Mechanical:MountingHole
Connections:
- wire segments 84 -> 89
Changed lines of the file:
@@
 $EndSheet
 $Sheet
-S 9500 2780 1500 920
+S 9500 3180 1500 920
 U 5FC5E24D
 F0 "SERVOS" 50
 F1 "SERVOS.sch" 50
-F2 "SERVO1" I L 9500 2900 50
-F3 "SERVO2" I L 9500 3050 50
-F4 "SERVO3" I L 9500 3200 50
-F5 "SERVO4" I L 9500 3350 50
-F6 "SERVO5" I L 9500 3500 50
-F7 "SERVO6" I L 9500 3650 50
-$EndSheet
-$Sheet
-S 9500 4170 1500 230
+F2 "SERVO1" I L 9500 3300 50
+F3 "SERVO2" I L 9500 3450 50
+F4 "SERVO3" I L 9500 3600 50
+F5 "SERVO4" I L 9500 3750 50
+F6 "SERVO5" I L 9500 3900 50
+F7 "SERVO6" I L 9500 4050 50
+$EndSheet
+$Sheet
+S 9500 4420 1500 230
 U 5FC6109B
 F0 "FANS" 50
 F1 "FANS.sch" 50
-F2 "FAN_CONTROL" I L 9500 4300 50
+F2 "FAN_CONTROL" I L 9500 4550 50
 $EndSheet
 Wire Wire Line
@@
 $EndSheet
 $Sheet
-S 9500 1550 1500 800
+S 9500 1550 1500 1200
 U 5FDA9108
 F0 "Barometer" 50
@@
 F5 "CSB" I L 9500 2100 50
 F6 "CS_BARO2" I L 9500 2250 50
+F7 "MOSI_2" I L 9500 2400 50
+F8 "SCK_2" I L 9500 2550 50
+F9 "MISO_2" I L 9500 2700 50
 $EndSheet
 Wire Wire Line
@@
 Wire Notes Line
 	8800 550  11100 550
-Wire Notes Line
-	11100 550  11100 2450
-Wire Notes Line
-	11100 2450 8800 2450
-Wire Notes Line
-	8800 2450 8800 550
-Text Notes 9750 2550 0    50   ~ 0
+Text Notes 9950 3000 0    50   ~ 0
 SENSORS\n
 Wire Notes Line
@@
 	650  7250 650  6500
 Wire Wire Line
-	9500 2900 8900 2900
-Wire Wire Line
-	9500 3050 8900 3050
-Wire Wire Line
-	9500 3200 8900 3200
-Wire Wire Line
-	9500 3350 8900 3350
-Text Label 9050 2900 0    50   ~ 0
+	9500 3300 8900 3300
+Wire Wire Line
+	9500 3450 8900 3450
+Wire Wire Line
+	9500 3600 8900 3600
+Wire Wire Line
+	9500 3750 8900 3750
+Text Label 9050 3300 0    50   ~ 0
 SERVO1
-Text Label 9050 3050 0    50   ~ 0
+Text Label 9050 3450 0    50   ~ 0
 SERVO2
-Text Label 9050 3200 0    50   ~ 0
+Text Label 9050 3600 0    50   ~ 0
 SERVO3
-Text Label 9050 3350 0    50   ~ 0
+Text Label 9050 3750 0    50   ~ 0
 SERVO4
 Wire Notes Line
-	8800 2650 11100 2650
-Text Notes 9800 3900 0    50   ~ 0
+	8800 3050 11100 3050
+Text Notes 9800 4300 0    50   ~ 0
 SERVOS\n
 Wire Wire Line
-	9500 4300 8900 4300
-Wire Notes Line
-	8800 4050 11100 4050
-Wire Notes Line
-	11100 4050 11100 4500
-Wire Notes Line
-	11100 4500 8800 4500
-Wire Notes Line
-	8800 4500 8800 4050
+	9500 4550 8900 4550
+Wire Notes Line
+	8800 4300 11100 4300
+Wire Notes Line
+	11100 4300 11100 4750
+Wire Notes Line
+	11100 4750 8800 4750
+Wire Notes Line
+	8800 4750 8800 4300
 Wire Wire Line
 	6950 850  7550 850
@@
 Text Label 7250 3050 0    50   ~ 0
 FANS
-Text Label 9100 4300 0    50   ~ 0
+Text Label 9100 4550 0    50   ~ 0
 FANS
 $Sheet
@@
 $EndSheet
 $Sheet
-S 9500 4750 1500 400
+S 9500 5000 1500 400
 U 60334804
 F0 "LED" 50
 F1 "LED.sch" 50
-F2 "LED_RED" I L 9500 4850 50
-F3 "LED_GREEN" I L 9500 4950 50
-F4 "LED_BLUE" I L 9500 5050 50
-$EndSheet
-Wire Wire Line
-	9500 4850 8900 4850
-Wire Wire Line
-	9500 4950 8900 4950
-Wire Wire Line
-	9500 5050 8900 5050
-Text Label 9050 4850 0    50   ~ 0
+F2 "LED_RED" I L 9500 5100 50
+F3 "LED_GREEN" I L 9500 5200 50
+F4 "LED_BLUE" I L 9500 5300 50
+$EndSheet
+Wire Wire Line
+	9500 5100 8900 5100
+Wire Wire Line
+	9500 5200 8900 5200
+Wire Wire Line
+	9500 5300 8900 5300
+Text Label 9050 5100 0    50   ~ 0
 LED_RED
-Text Label 9050 4950 0    50   ~ 0
+Text Label 9050 5200 0    50   ~ 0
 LED_GREEN
-Text Label 9050 5050 0    50   ~ 0
+Text Label 9050 5300 0    50   ~ 0
 LED_BLUE
 Wire Notes Line
-	8800 5250 11100 5250
-Wire Notes Line
-	11100 5250 11100 4650
-Wire Notes Line
-	11100 4650 8800 4650
-Wire Notes Line
-	8800 4650 8800 5250
-Text Notes 9800 5350 0    50   ~ 0
+	8800 5500 11100 5500
+Wire Notes Line
+	11100 5500 11100 4900
+Wire Notes Line
+	11100 4900 8800 4900
+Wire Notes Line
+	8800 4900 8800 5500
+Text Notes 9800 5600 0    50   ~ 0
 LED\n
-Text Notes 9850 4600 0    50   ~ 0
+Text Notes 9850 4850 0    50   ~ 0
 FANS\n
 $Sheet
-S 9500 5550 1500 500
+S 9500 5800 1500 500
 U 60353E60
 F0 "FLASH" 50
 F1 "FLASH.sch" 50
-F2 "CS_FLASH" I L 9500 5650 50
-F3 "SCLK" I L 9500 5750 50
-F4 "MOSI" I L 9500 5850 50
-F5 "MISO" I L 9500 5950 50
-$EndSheet
-Wire Wire Line
-	9500 5650 8900 5650
-Wire Wire Line
-	9500 5750 8900 5750
-Wire Wire Line
-	9500 5850 8900 5850
-Wire Wire Line
-	9500 5950 8900 5950
-Text Label 9050 5650 0    50   ~ 0
+F2 "CS_FLASH" I L 9500 5900 50
+F3 "SCLK" I L 9500 6000 50
+F4 "MOSI" I L 9500 6100 50
+F5 "MISO" I L 9500 6200 50
+$EndSheet
+Wire Wire Line
+	9500 5900 8900 5900
+Wire Wire Line
+	9500 6000 8900 6000
+Wire Wire Line
+	9500 6100 8900 6100
+Wire Wire Line
+	9500 6200 8900 6200
+Text Label 9050 5900 0    50   ~ 0
 CS_FLASH
-Text Label 9050 5750 0    50   ~ 0
+Text Label 9050 6000 0    50   ~ 0
 SCK
-Text Label 9050 5850 0    50   ~ 0
+Text Label 9050 6100 0    50   ~ 0
 MOSI
-Text Label 9050 5950 0    50   ~ 0
+Text Label 9050 6200 0    50   ~ 0
 MISO
 Wire Notes Line
-	8800 5400 8800 6150
-Wire Notes Line
-	8800 6150 11100 6150
-Wire Notes Line
-	11100 6150 11100 5400
-Wire Notes Line
-	11100 5400 8800 5400
-Text Notes 9750 6350 0    50   ~ 0
+	8800 5650 8800 6400
+Wire Notes Line
+	8800 6400 11100 6400
+Wire Notes Line
+	11100 6400 11100 5650
+Wire Notes Line
+	11100 5650 8800 5650
+Text Notes 9750 6600 0    50   ~ 0
 FLASH\n\n
 $Sheet
@@
 F22 "PWM3" I R 6950 3400 50
 F23 "PWM4" I R 6950 3500 50
+F24 "FLASH_CS" I R 6950 3600 50
+F25 "SD_FLASH" I R 6950 4000 50
 $EndSheet
 Wire Wire Line
@@
 LED_BLUE
 Wire Wire Line
-	9500 3500 8900 3500
-Wire Wire Line
-	9500 3650 8900 3650
-Text Label 9050 3500 0    50   ~ 0
+	9500 3900 8900 3900
+Wire Wire Line
+	9500 4050 8900 4050
+Text Label 9050 3900 0    50   ~ 0
 SERVO5
-Text Label 9050 3650 0    50   ~ 0
+Text Label 9050 4050 0    50   ~ 0
 SERVO6
 Wire Notes Line
-	11100 3800 8800 3800
-Wire Notes Line
-	11100 2650 11100 3800
-Wire Notes Line
-	8800 2650 8800 3800
+	11100 4200 8800 4200
+Wire Notes Line
+	11100 3050 11100 4200
+Wire Notes Line
+	8800 3050 8800 4200
 Wire Wire Line
 	6950 3200 7650 3200
@@
 Wire Wire Line
 	6950 3500 7650 3500
+Text Label 7200 3400 0    50   ~ 0
+CS_BARO
+Text Label 7200 3500 0    50   ~ 0
+CS_BARO2
+Wire Wire Line
+	6950 3600 7650 3600
+Text Label 7200 3600 0    50   ~ 0
+CS_FLASH
+Wire Notes Line
+	11100 2850 8800 2850
+Wire Notes Line
+	11100 550  11100 2850
+Wire Notes Line
+	8800 550  8800 2850
+Wire Wire Line
+	9500 2400 8900 2400
+Wire Wire Line
+	9500 2550 8900 2550
+Wire Wire Line
+	9500 2700 8900 2700
+Text Label 9100 2400 0    50   ~ 0
+MOSI
+Text Label 9100 2550 0    50   ~ 0
+SCK
+Text Label 9100 2700 0    50   ~ 0
+MISO
+Wire Wire Line
+	6950 4000 7650 4000
+Text Label 7200 4000 0    50   ~ 0
+CS_SD
+$Comp
+L Mechanical:MountingHole H101
+U 1 1 6050C077
+P 5250 4700
+F 0 "H101" H 5350 4746 50  0000 L CNN
+F 1 "MountingHole" H 5350 4655 50  0000 L CNN
+F 2 "MountingHole:MountingHole_3.2mm_M3" H 5250 4700 50  0001 C CNN
+F 3 "~" H 5250 4700 50  0001 C CNN
+	1    5250 4700
+	1    0    0    -1
+$EndComp
+$Comp
+L Mechanical:MountingHole H102
+U 1 1 6050ECED
+P 5250 4900
+F 0 "H102" H 5350 4946 50  0000 L CNN
+F 1 "MountingHole" H 5350 4855 50  0000 L CNN
+F 2 "MountingHole:MountingHole_3.2mm_M3" H 5250 4900 50  0001 C CNN
+F 3 "~" H 5250 4900 50  0001 C CNN
+	1    5250 4900
+	1    0    0    -1
+$EndComp
+$Comp
+L Mechanical:MountingHole H103
+U 1 1 6050EE4F
+P 5250 5100
+F 0 "H103" H 5350 5146 50  0000 L CNN
+F 1 "MountingHole" H 5350 5055 50  0000 L CNN
+F 2 "MountingHole:MountingHole_3.2mm_M3" H 5250 5100 50  0001 C CNN
+F 3 "~" H 5250 5100 50  0001 C CNN
+	1    5250 5100
+	1    0    0    -1
+$EndComp
+$Comp
+L Mechanical:MountingHole H104
+U 1 1 6050F089
+P 5250 5300
+F 0 "H104" H 5350 5346 50  0000 L CNN
+F 1 "MountingHole" H 5350 5255 50  0000 L CNN
+F 2 "MountingHole:MountingHole_3.2mm_M3" H 5250 5300 50  0001 C CNN
+F 3 "~" H 5250 5300 50  0001 C CNN
+	1    5250 5300
+	1    0    0    -1
+$EndComp
 $EndSCHEMATC
