File: hardware/Payload_Computer/Rev 2/POWER REGULATION.sch (KiCad schematic (older format))
At the start: 4 parts

Commit message: Minor Updates
Parts:
- gave numbers to parts that had none: 4
Changed lines of the file:
@@
 $EndDescr
 $Comp
-L power:+5V #PWR?
+L power:+5V #PWR0106
 U 1 1 6056925C
 P 7250 1600
-F 0 "#PWR?" H 7250 1450 50  0001 C CNN
+F 0 "#PWR0106" H 7250 1450 50  0001 C CNN
 F 1 "+5V" V 7265 1728 50  0000 L CNN
 F 2 "" H 7250 1600 50  0001 C CNN
@@
 NoConn ~ 6900 1500
 $Comp
-L power:+BATT #PWR?
+L power:+BATT #PWR0107
 U 1 1 6056987F
 P 4400 1500
-F 0 "#PWR?" H 4400 1350 50  0001 C CNN
+F 0 "#PWR0107" H 4400 1350 50  0001 C CNN
 F 1 "+BATT" V 4415 1627 50  0000 L CNN
 F 2 "" H 4400 1500 50  0001 C CNN
@@
 	4400 1600 4700 1600
 $Comp
-L power:GND #PWR?
+L power:GND #PWR0108
 U 1 1 60568D35
 P 4400 1600
-F 0 "#PWR?" H 4400 1350 50  0001 C CNN
+F 0 "#PWR0108" H 4400 1350 50  0001 C CNN
 F 1 "GND" V 4405 1472 50  0000 R CNN
 F 2 "" H 4400 1600 50  0001 C CNN
@@
 $EndComp
 $Comp
-L 2021-03-20_20-22-22:MIC29151-5.0WU-TR U?
+L 2021-03-20_20-22-22:MIC29151-5.0WU-TR U301
 U 1 1 60567CDA
 P 4700 1400
-F 0 "U?" H 5800 1788 60  0000 C CNN
+F 0 "U301" H 5800 1788 60  0000 C CNN
 F 1 "MIC29151-5.0WU-TR" H 5800 1682 60  0000 C CNN
 F 2 "footprints:MIC29151-5.0WU-TR" H 5800 1640 60  0001 C CNN
@@
 $EndComp
 $Comp
-L power:GND #PWR?
+L power:GND #PWR0109
 U 1 1 6056AAC6
 P 7300 1400
-F 0 "#PWR?" H 7300 1150 50  0001 C CNN
+F 0 "#PWR0109" H 7300 1150 50  0001 C CNN
 F 1 "GND" V 7305 1272 50  0000 R CNN
 F 2 "" H 7300 1400 50  0001 C CNN
@@
 	7900 1750 7900 1450
 $Comp
-L power:GND #PWR?
+L power:GND #PWR0110
 U 1 1 6056FC7A
 P 7900 1750
-F 0 "#PWR?" H 7900 1500 50  0001 C CNN
+F 0 "#PWR0110" H 7900 1500 50  0001 C CNN
 F 1 "GND" V 7905 1622 50  0000 R CNN
 F 2 "" H 7900 1750 50  0001 C CNN
@@
 $EndComp
 $Comp
-L Device:CP1 C?
+L Device:CP1 C302
 U 1 1 6056FC80
 P 7900 1300
-F 0 "C?" H 8015 1346 50  0000 L CNN
+F 0 "C302" H 8015 1346 50  0000 L CNN
 F 1 "10uF" H 8015 1255 50  0000 L CNN
 F 2 "Capacitor_Tantalum_SMD:CP_EIA-6032-20_AVX-F_Pad2.25x2.35mm_HandSolder" H 7900 1300 50  0001 C CNN
@@
 $EndComp
 $Comp
-L power:+5V #PWR?
+L power:+5V #PWR0111
 U 1 1 6056FE27
 P 7900 950
-F 0 "#PWR?" H 7900 800 50  0001 C CNN
+F 0 "#PWR0111" H 7900 800 50  0001 C CNN
 F 1 "+5V" H 7915 1123 50  0000 C CNN
 F 2 "" H 7900 950 50  0001 C CNN
@@
 	2650 1650 2650 1350
 $Comp
-L power:GND #PWR?
+L power:GND #PWR0112
 U 1 1 60571464
 P 2650 1650
-F 0 "#PWR?" H 2650 1400 50  0001 C CNN
+F 0 "#PWR0112" H 2650 1400 50  0001 C CNN
 F 1 "GND" V 2655 1522 50  0000 R CNN
 F 2 "" H 2650 1650 50  0001 C CNN
@@
 $EndComp
 $Comp
-L Device:CP1 C?
+L Device:CP1 C301
 U 1 1 6057146B
 P 2650 1200
-F 0 "C?" H 2765 1246 50  0000 L CNN
+F 0 "C301" H 2765 1246 50  0000 L CNN
 F 1 "10uF" H 2765 1155 50  0000 L CNN
 F 2 "Capacitor_Tantalum_SMD:CP_EIA-6032-20_AVX-F_Pad2.25x2.35mm_HandSolder" H 2650 1200 50  0001 C CNN
@@
 $EndComp
 $Comp
-L power:+BATT #PWR?
+L power:+BATT #PWR0113
 U 1 1 6057154B
 P 2650 850
-F 0 "#PWR?" H 2650 700 50  0001 C CNN
+F 0 "#PWR0113" H 2650 700 50  0001 C CNN
 F 1 "+BATT" H 2665 1023 50  0000 C CNN
 F 2 "" H 2650 850 50  0001 C CNN
@@
 $EndComp
 $Comp
-L Device:D D?
+L Device:D D301
 U 1 1 60572F10
 P 3750 1500
-F 0 "D?" H 3750 1283 50  0000 C CNN
+F 0 "D301" H 3750 1283 50  0000 C CNN
 F 1 "D" H 3750 1374 50  0000 C CNN
 F 2 "" H 3750 1500 50  0001 C CNN

Commit message: Finished the overbuilt power supply and did some minor routing
Parts:
- removed D301: D, symbol Device:D
- added C303, C304: 10uF, Capacitor_Tantalum_SMD:CP_EIA-6032-20_AVX-F_Pad2.25x2.35mm_HandSolder, symbol Device:CP1
- added CR301, CR302: B320B-13, footprints-diode:B320B-13, symbol 2021-03-23_04-45-24:B320B-13
- added VR301: LT1963AEST-3.3#PBF, LT1963AEST-3:SOT223, symbol LT1963AEST-3.3_PBF:LT1963AEST-3.3#PBF
Connections:
- net labels added: +3.3V
- wire segments 11 -> 25
Other:
- note added: "3.3V REGULATOR\n"
- moved on the sheet: C301
Changed lines of the file:
@@
 L power:+BATT #PWR0107
 U 1 1 6056987F
-P 4400 1500
-F 0 "#PWR0107" H 4400 1350 50  0001 C CNN
-F 1 "+BATT" V 4415 1627 50  0000 L CNN
-F 2 "" H 4400 1500 50  0001 C CNN
-F 3 "" H 4400 1500 50  0001 C CNN
-	1    4400 1500
+P 3350 1500
+F 0 "#PWR0107" H 3350 1350 50  0001 C CNN
+F 1 "+BATT" V 3365 1627 50  0000 L CNN
+F 2 "" H 3350 1500 50  0001 C CNN
+F 3 "" H 3350 1500 50  0001 C CNN
+	1    3350 1500
 	0    -1   -1   0
 $EndComp
-Wire Wire Line
-	4400 1500 4500 1500
 Wire Wire Line
 	4700 1400 4500 1400
@@
 $EndComp
 Wire Wire Line
-	2650 850  2650 1050
-Wire Wire Line
-	2650 1650 2650 1350
+	4300 1500 4300 1300
 $Comp
 L power:GND #PWR0112
 U 1 1 60571464
-P 2650 1650
-F 0 "#PWR0112" H 2650 1400 50  0001 C CNN
-F 1 "GND" V 2655 1522 50  0000 R CNN
-F 2 "" H 2650 1650 50  0001 C CNN
-F 3 "" H 2650 1650 50  0001 C CNN
-	1    2650 1650
-	1    0    0    -1
+P 4300 800
+F 0 "#PWR0112" H 4300 550 50  0001 C CNN
+F 1 "GND" V 4305 672 50  0000 R CNN
+F 2 "" H 4300 800 50  0001 C CNN
+F 3 "" H 4300 800 50  0001 C CNN
+	1    4300 800
+	-1   0    0    1
 $EndComp
 $Comp
 L Device:CP1 C301
 U 1 1 6057146B
-P 2650 1200
-F 0 "C301" H 2765 1246 50  0000 L CNN
-F 1 "10uF" H 2765 1155 50  0000 L CNN
-F 2 "Capacitor_Tantalum_SMD:CP_EIA-6032-20_AVX-F_Pad2.25x2.35mm_HandSolder" H 2650 1200 50  0001 C CNN
-F 3 "https://www.vishay.com/docs/40002/293d.pdf" H 2650 1200 50  0001 C CNN
-F 4 "718-1958-1-ND" H 2650 1200 50  0001 C CNN "DIGIKEY"
-	1    2650 1200
-	1    0    0    -1
-$EndComp
-$Comp
-L power:+BATT #PWR0113
-U 1 1 6057154B
-P 2650 850
-F 0 "#PWR0113" H 2650 700 50  0001 C CNN
-F 1 "+BATT" H 2665 1023 50  0000 C CNN
-F 2 "" H 2650 850 50  0001 C CNN
-F 3 "" H 2650 850 50  0001 C CNN
-	1    2650 850
-	1    0    0    -1
-$EndComp
-$Comp
-L Device:D D301
-U 1 1 60572F10
-P 3750 1500
-F 0 "D301" H 3750 1283 50  0000 C CNN
-F 1 "D" H 3750 1374 50  0000 C CNN
-F 2 "" H 3750 1500 50  0001 C CNN
-F 3 "~" H 3750 1500 50  0001 C CNN
-	1    3750 1500
-	-1   0    0    1
-$EndComp
+P 4300 1150
+F 0 "C301" H 4415 1196 50  0000 L CNN
+F 1 "10uF" H 4415 1105 50  0000 L CNN
+F 2 "Capacitor_Tantalum_SMD:CP_EIA-6032-20_AVX-F_Pad2.25x2.35mm_HandSolder" H 4300 1150 50  0001 C CNN
+F 3 "https://www.vishay.com/docs/40002/293d.pdf" H 4300 1150 50  0001 C CNN
+F 4 "718-1958-1-ND" H 4300 1150 50  0001 C CNN "DIGIKEY"
+	1    4300 1150
+	-1   0    0    1
+$EndComp
+$Comp
+L LT1963AEST-3.3_PBF:LT1963AEST-3.3#PBF VR301
+U 1 1 605971F7
+P 5400 3300
+F 0 "VR301" H 5750 3870 50  0000 C CNN
+F 1 "LT1963AEST-3.3#PBF" H 5750 3779 50  0000 C CNN
+F 2 "LT1963AEST-3:SOT223" H 5400 3300 50  0001 L BNN
+F 3 "" H 5400 3300 50  0001 L BNN
+F 4 "LT1963AEST-3.3#PBF" H 5400 3300 50  0001 L BNN "MPN"
+F 5 "Linear Technology" H 5400 3300 50  0001 L BNN "MANUFACTURER"
+F 6 "LT1963AEST-3.3#PBF-ND" H 5400 3300 50  0001 C CNN "Digikey"
+	1    5400 3300
+	1    0    0    -1
+$EndComp
+$Comp
+L power:+BATT #PWR0303
+U 1 1 60597F5E
+P 4050 3000
+F 0 "#PWR0303" H 4050 2850 50  0001 C CNN
+F 1 "+BATT" V 4065 3127 50  0000 L CNN
+F 2 "" H 4050 3000 50  0001 C CNN
+F 3 "" H 4050 3000 50  0001 C CNN
+	1    4050 3000
+	0    -1   -1   0
+$EndComp
+$Comp
+L power:GND #PWR0304
+U 1 1 60598D50
+P 4900 3200
+F 0 "#PWR0304" H 4900 2950 50  0001 C CNN
+F 1 "GND" V 4905 3072 50  0000 R CNN
+F 2 "" H 4900 3200 50  0001 C CNN
+F 3 "" H 4900 3200 50  0001 C CNN
+	1    4900 3200
+	0    1    1    0
+$EndComp
+Wire Wire Line
+	5200 3200 5000 3200
+Wire Wire Line
+	5200 3100 5000 3100
+Wire Wire Line
+	5000 3100 5000 3200
+Connection ~ 5000 3200
+Wire Wire Line
+	5000 3200 4900 3200
+$Comp
+L power:+3.3V #PWR0305
+U 1 1 60599C96
+P 6600 3000
+F 0 "#PWR0305" H 6600 2850 50  0001 C CNN
+F 1 "+3.3V" V 6615 3128 50  0000 L CNN
+F 2 "" H 6600 3000 50  0001 C CNN
+F 3 "" H 6600 3000 50  0001 C CNN
+	1    6600 3000
+	0    1    1    0
+$EndComp
+Wire Wire Line
+	6300 3000 6600 3000
+Wire Wire Line
+	4000 1500 4300 1500
+Wire Wire Line
+	3350 1500 3600 1500
+Wire Wire Line
+	5100 3000 5100 2800
+Wire Wire Line
+	5100 2200 5100 2500
+$Comp
+L power:GND #PWR0302
+U 1 1 6059D143
+P 5100 2200
+F 0 "#PWR0302" H 5100 1950 50  0001 C CNN
+F 1 "GND" V 5105 2072 50  0000 R CNN
+F 2 "" H 5100 2200 50  0001 C CNN
+F 3 "" H 5100 2200 50  0001 C CNN
+	1    5100 2200
+	-1   0    0    1
+$EndComp
+$Comp
+L Device:CP1 C303
+U 1 1 6059D14A
+P 5100 2650
+F 0 "C303" H 5215 2696 50  0000 L CNN
+F 1 "10uF" H 5215 2605 50  0000 L CNN
+F 2 "Capacitor_Tantalum_SMD:CP_EIA-6032-20_AVX-F_Pad2.25x2.35mm_HandSolder" H 5100 2650 50  0001 C CNN
+F 3 "https://www.vishay.com/docs/40002/293d.pdf" H 5100 2650 50  0001 C CNN
+F 4 "718-1958-1-ND" H 5100 2650 50  0001 C CNN "DIGIKEY"
+	1    5100 2650
+	-1   0    0    1
+$EndComp
+Wire Wire Line
+	7900 2650 7900 2850
+Wire Wire Line
+	7900 3450 7900 3150
+$Comp
+L power:GND #PWR0307
+U 1 1 6059DE65
+P 7900 3450
+F 0 "#PWR0307" H 7900 3200 50  0001 C CNN
+F 1 "GND" V 7905 3322 50  0000 R CNN
+F 2 "" H 7900 3450 50  0001 C CNN
+F 3 "" H 7900 3450 50  0001 C CNN
+	1    7900 3450
+	1    0    0    -1
+$EndComp
+$Comp
+L Device:CP1 C304
+U 1 1 6059DE6C
+P 7900 3000
+F 0 "C304" H 8015 3046 50  0000 L CNN
+F 1 "10uF" H 8015 2955 50  0000 L CNN
+F 2 "Capacitor_Tantalum_SMD:CP_EIA-6032-20_AVX-F_Pad2.25x2.35mm_HandSolder" H 7900 3000 50  0001 C CNN
+F 3 "https://www.vishay.com/docs/40002/293d.pdf" H 7900 3000 50  0001 C CNN
+F 4 "718-1958-1-ND" H 7900 3000 50  0001 C CNN "DIGIKEY"
+	1    7900 3000
+	1    0    0    -1
+$EndComp
+$Comp
+L power:+3.3V #PWR0306
+U 1 1 6059E119
+P 7900 2650
+F 0 "#PWR0306" H 7900 2500 50  0001 C CNN
+F 1 "+3.3V" H 7915 2823 50  0000 C CNN
+F 2 "" H 7900 2650 50  0001 C CNN
+F 3 "" H 7900 2650 50  0001 C CNN
+	1    7900 2650
+	1    0    0    -1
+$EndComp
+Text Notes 5450 2600 0    50   ~ 0
+3.3V REGULATOR\n
+$Comp
+L 2021-03-23_04-45-24:B320B-13 CR301
+U 1 1 605A0D52
+P 3600 1500
+F 0 "CR301" H 3800 1763 60  0000 C CNN
+F 1 "B320B-13" H 3800 1657 60  0000 C CNN
+F 2 "footprints-diode:B320B-13" H 3800 1140 60  0001 C CNN
+F 3 "https://media.digikey.com/pdf/Data%20Sheets/Diodes%20PDFs/B320B-B360B_Rev10-2.pdf" H 3800 1657 60  0001 C CNN
+F 4 "B320B-FDICT-ND" H 3600 1500 50  0001 C CNN "DIGIKEY"
+	1    3600 1500
+	1    0    0    -1
+$EndComp
+Wire Wire Line
+	4050 3000 4350 3000
+$Comp
+L 2021-03-23_04-45-24:B320B-13 CR302
+U 1 1 605A362B
+P 4350 3000
+F 0 "CR302" H 4550 3263 60  0000 C CNN
+F 1 "B320B-13" H 4550 3157 60  0000 C CNN
+F 2 "footprints-diode:B320B-13" H 4550 2640 60  0001 C CNN
+F 3 "https://media.digikey.com/pdf/Data%20Sheets/Diodes%20PDFs/B320B-B360B_Rev10-2.pdf" H 4550 3157 60  0001 C CNN
+F 4 "B320B-FDICT-ND" H 4350 3000 50  0001 C CNN "DIGIKEY"
+	1    4350 3000
+	1    0    0    -1
+$EndComp
+Connection ~ 4300 1500
+Wire Wire Line
+	4300 1500 4500 1500
+Wire Wire Line
+	4300 800  4300 1000
+Connection ~ 5100 3000
+Wire Wire Line
+	5100 3000 5200 3000
+Wire Wire Line
+	4750 3000 5100 3000
 $EndSCHEMATC

Commit message: I did something
Parts:
- VR301: MANUFACTURER Linear Technology -> No
Changed lines of the file:
@@
 F 3 "" H 5400 3300 50  0001 L BNN
 F 4 "LT1963AEST-3.3#PBF" H 5400 3300 50  0001 L BNN "MPN"
-F 5 "Linear Technology" H 5400 3300 50  0001 L BNN "MANUFACTURER"
+F 5 "No" H 5400 3300 50  0001 L BNN "MANUFACTURER"
 F 6 "LT1963AEST-3.3#PBF-ND" H 5400 3300 50  0001 C CNN "Digikey"
 	1    5400 3300
