File: hardware/Payload_Computer/Rev 2/FLASH CHIP.sch (KiCad schematic (older format))
At the start: 1 part, among them U701 W25N01GVZEIG

Commit message: Finished some routing
Parts:
- added C701: 100nF, Capacitor_SMD:C_0603_1608Metric_Pad1.08x0.95mm_HandSolder, symbol Device:C
Connections:
- net +3V3: now also C701.1
- net GND: now also C701.2
- net MISO: now also U701.2 (DOIO1)
- net MOSI: now also U701.5 (DIIO0)
Changed lines of the file:
@@
 Text HLabel 7850 3800 2    50   Input ~ 0
 MOSI
+Wire Wire Line
+	7850 3800 7350 3800
+Wire Wire Line
+	4450 3500 4950 3500
+$Comp
+L Device:C C701
+U 1 1 60727D9F
+P 9050 3050
+F 0 "C701" H 9165 3096 50  0000 L CNN
+F 1 "100nF" H 9165 3005 50  0000 L CNN
+F 2 "Capacitor_SMD:C_0603_1608Metric_Pad1.08x0.95mm_HandSolder" H 9088 2900 50  0001 C CNN
+F 3 "~" H 9050 3050 50  0001 C CNN
+	1    9050 3050
+	1    0    0    -1
+$EndComp
+$Comp
+L power:+3.3V #PWR0118
+U 1 1 607281EE
+P 9050 2750
+F 0 "#PWR0118" H 9050 2600 50  0001 C CNN
+F 1 "+3.3V" V 9065 2878 50  0000 L CNN
+F 2 "" H 9050 2750 50  0001 C CNN
+F 3 "" H 9050 2750 50  0001 C CNN
+	1    9050 2750
+	1    0    0    -1
+$EndComp
+$Comp
+L power:GND #PWR0119
+U 1 1 607287AA
+P 9050 3400
+F 0 "#PWR0119" H 9050 3150 50  0001 C CNN
+F 1 "GND" V 9055 3272 50  0000 R CNN
+F 2 "" H 9050 3400 50  0001 C CNN
+F 3 "" H 9050 3400 50  0001 C CNN
+	1    9050 3400
+	1    0    0    -1
+$EndComp
+Wire Wire Line
+	9050 2750 9050 2900
+Wire Wire Line
+	9050 3200 9050 3400
 $EndSCHEMATC
