File: hardware/Payload_Computer/Rev 2/SD_CARD.sch (KiCad schematic (older format))
At the start: 1 part

Commit message: Did some stuff
Parts:
- gave numbers to parts that had none: 1
Changed lines of the file:
@@
 $Descr A4 11693 8268
 encoding utf-8
-Sheet 6 6
+Sheet 6 7
 Title ""
 Date ""
@@
 $EndDescr
 $Comp
-L 2021-04-03_19-33-36:503182-1852 U?
+L 2021-04-03_19-33-36:503182-1852 U601
 U 1 1 606A8D60
 P 4550 3500
-F 0 "U?" H 5550 3887 60  0000 C CNN
+F 0 "U601" H 5550 3887 60  0000 C CNN
 F 1 "503182-1852" H 5550 3781 60  0000 C CNN
 F 2 "SD_CARD:503182-1852" H 5550 3740 60  0001 C CNN
@@
 $EndComp
 $Comp
-L power:+3.3V #PWR?
+L power:+3.3V #PWR0601
 U 1 1 606A97F8
 P 4250 3800
-F 0 "#PWR?" H 4250 3650 50  0001 C CNN
+F 0 "#PWR0601" H 4250 3650 50  0001 C CNN
 F 1 "+3.3V" V 4265 3928 50  0000 L CNN
 F 2 "" H 4250 3800 50  0001 C CNN
@@
 $EndComp
 $Comp
-L power:GND #PWR?
+L power:GND #PWR0602
 U 1 1 606AA80F
 P 6800 3700
-F 0 "#PWR?" H 6800 3450 50  0001 C CNN
+F 0 "#PWR0602" H 6800 3450 50  0001 C CNN
 F 1 "GND" V 6805 3572 50  0000 R CNN
 F 2 "" H 6800 3700 50  0001 C CNN

Commit message: Finished some routing
Parts:
- added C601: 100nF, Capacitor_SMD:C_0603_1608Metric_Pad1.08x0.95mm_HandSolder, symbol Device:C
Connections:
- net +3V3: now also C601.1
- net GND: now also C601.2
Changed lines of the file:
@@
 	6550 3700 6800 3700
 Wire Wire Line
-	4550 3800 4250 3800
+	4550 3800 4400 3800
 Text HLabel 6800 3800 2    50   Input ~ 0
 SCK
@@
 	6800 3600 6550 3600
 NoConn ~ 6550 3500
+$Comp
+L Device:C C601
+U 1 1 60726DB3
+P 4400 3950
+F 0 "C601" H 4515 3996 50  0000 L CNN
+F 1 "100nF" H 4515 3905 50  0000 L CNN
+F 2 "Capacitor_SMD:C_0603_1608Metric_Pad1.08x0.95mm_HandSolder" H 4438 3800 50  0001 C CNN
+F 3 "~" H 4400 3950 50  0001 C CNN
+	1    4400 3950
+	1    0    0    -1
+$EndComp
+Connection ~ 4400 3800
+Wire Wire Line
+	4400 3800 4250 3800
+$Comp
+L power:GND #PWR0117
+U 1 1 607272DF
+P 4400 4300
+F 0 "#PWR0117" H 4400 4050 50  0001 C CNN
+F 1 "GND" V 4405 4172 50  0000 R CNN
+F 2 "" H 4400 4300 50  0001 C CNN
+F 3 "" H 4400 4300 50  0001 C CNN
+	1    4400 4300
+	1    0    0    -1
+$EndComp
+Wire Wire Line
+	4400 4300 4400 4100
 $EndSCHEMATC
