File: hardware/Payload_Computer/Rev 2/TEENSY3.sch (KiCad schematic (older format))
At the start: 1 part, among them U201 Teensy3.2

Commit message: More routing and added BNO055
Connections:
- net SCL: now reaches U201.25 (18_A4_SDA0_Touch)
- net SDA: now reaches U201.26 (19_A5_SCL0_Touch)
Changed lines of the file:
@@
 $Descr A4 11693 8268
 encoding utf-8
-Sheet 2 3
+Sheet 2 5
 Title ""
 Date ""
@@
 Wire Wire Line
 	6950 4700 7450 4700
+Text HLabel 4500 4800 0    50   Input ~ 0
+SCL
+Wire Wire Line
+	4500 4800 4950 4800
+Text HLabel 4500 4900 0    50   Input ~ 0
+SDA
+Wire Wire Line
+	4500 4900 4950 4900
 $EndSCHEMATC

Commit message: Did some stuff
Connections:
- net MOSI: now reaches U201.13 (11_DOUT)
- net MISO: now reaches U201.14 (12_DIN)
- net SCK: now reaches U201.20 (13_LED_SCK)
Changed lines of the file:
@@
 $Descr A4 11693 8268
 encoding utf-8
-Sheet 2 6
+Sheet 2 7
 Title ""
 Date ""
@@
 Wire Wire Line
 	4500 4900 4950 4900
+Text HLabel 4500 4300 0    50   Input ~ 0
+SCK
+Text HLabel 4500 3600 0    50   Input ~ 0
+MOSI
+Text HLabel 4500 3700 0    50   Input ~ 0
+MISO
+Wire Wire Line
+	4500 3600 4950 3600
+Wire Wire Line
+	4500 3700 4950 3700
+Wire Wire Line
+	4500 4300 4950 4300
 $EndSCHEMATC

Commit message: Finished some routing
Connections:
- net SD_CS: now reaches U201.21 (14_A0_SCK)
- net FLASH_CS: now reaches U201.22 (15_A1_CS_Touch)
Changed lines of the file:
@@
 Wire Wire Line
 	4500 4300 4950 4300
+Text HLabel 4500 4400 0    50   Input ~ 0
+SD_CS
+Text HLabel 4500 4500 0    50   Input ~ 0
+FLASH_CS
+Wire Wire Line
+	4500 4400 4950 4400
+Wire Wire Line
+	4950 4500 4500 4500
 $EndSCHEMATC
